File: _saved_rangefinder.sch (KiCad schematic (older format))
At the start: 5 parts, among them U9 VL53L0X

Commit message: a few more footprints
Parts:
- U9: footprint (none) -> LGA12R50P4X4_200X200X86:LGA12R50P4X4_200X200X86
Changed lines of the file:
@@
 F 0 "U9" H 5600 4250 60  0000 C CNN
 F 1 "VL53L0X" H 5100 4250 60  0000 C CNN
-F 2 "" H 5350 3650 60  0001 C CNN
+F 2 "LGA12R50P4X4_200X200X86:LGA12R50P4X4_200X200X86" H 5350 3650 60  0001 C CNN
 F 3 "" H 5350 3650 60  0000 C CNN
 	1    5300 3700
