File: hdmi.sch (KiCad schematic (older format))
At the start: 31 parts, among them J5 MICRO_HDMI, U1 xc7a50tftg256, U11 GTL2002, U12 NC7WZ07P6X, U13 NC7SZ125M5X, U14 ADP198ACPZ-R7

Commit message: resolved ERC errors, and began assigning footprints
Parts:
- added C126: 100nF, Capacitors_SMD:C_0603, symbol C_Small
- added X1: KC5032A, symbol KC5032A
- C106, C107, C112, C113, C114, C115, C117: footprint (none) -> Capacitors_SMD:C_0603
- C109: footprint (none) -> Capacitors_SMD:C_1210
- C110, C111: footprint (none) -> Capacitors_SMD:C_0805
- C116: footprint (none) -> Capacitors_SMD:C_0402
- U11: footprint SO8N -> (none)
Connections:
- net labels added: CLK100MHz
- net labels removed: 3V3
- wire segments 134 -> 145
- no-connect marks 38 -> 37

Commit message: finished assigning cap footprints
Parts:
- C108: footprint (none) -> Capacitors_SMD:C_0603
Changed lines of the file:
@@
 	1950 4050 3950 4050
 $Comp
-L GND #PWR0117
+L GND #PWR120
 U 1 1 58643EDD
 P 2950 6900
-F 0 "#PWR0117" H 2950 6650 50  0001 C CNN
+F 0 "#PWR120" H 2950 6650 50  0001 C CNN
 F 1 "GND" H 2950 6750 50  0000 C CNN
 F 2 "" H 2950 6900 50  0000 C CNN
@@
 F 0 "C108" H 2525 6400 50  0000 L CNN
 F 1 "1nF, 250V" V 2350 6150 50  0000 L CNN
-F 2 "" H 2538 6150 50  0001 C CNN
+F 2 "Capacitors_SMD:C_0603" H 2538 6150 50  0001 C CNN
 F 3 "" H 2500 6300 50  0000 C CNN
 	1    2500 6300
@@
 Connection ~ 2150 6300
 $Comp
-L GND #PWR0118
+L GND #PWR118
 U 1 1 58644254
 P 2300 5300
-F 0 "#PWR0118" H 2300 5050 50  0001 C CNN
+F 0 "#PWR118" H 2300 5050 50  0001 C CNN
 F 1 "GND" H 2300 5150 50  0000 C CNN
 F 2 "" H 2300 5300 50  0000 C CNN
@@
 $EndComp
 $Comp
-L GND #PWR0119
+L GND #PWR117
 U 1 1 58644E40
 P 1800 2450
-F 0 "#PWR0119" H 1800 2200 50  0001 C CNN
+F 0 "#PWR117" H 1800 2200 50  0001 C CNN
 F 1 "GND" H 1800 2300 50  0000 C CNN
 F 2 "" H 1800 2450 50  0000 C CNN
@@
 Connection ~ 8800 3700
 $Comp
-L GND #PWR0120
+L GND #PWR127
 U 1 1 586484F8
 P 8800 3850
-F 0 "#PWR0120" H 8800 3600 50  0001 C CNN
+F 0 "#PWR127" H 8800 3600 50  0001 C CNN
 F 1 "GND" H 8800 3700 50  0000 C CNN
 F 2 "" H 8800 3850 50  0000 C CNN
@@
 Connection ~ 3350 5650
 $Comp
-L GND #PWR0121
+L GND #PWR122
 U 1 1 58662B25
 P 4450 5300
-F 0 "#PWR0121" H 4450 5050 50  0001 C CNN
+F 0 "#PWR122" H 4450 5050 50  0001 C CNN
 F 1 "GND" H 4450 5150 50  0000 C CNN
 F 2 "" H 4450 5300 50  0000 C CNN
@@
 Connection ~ 4750 7250
 $Comp
-L GND #PWR0122
+L GND #PWR121
 U 1 1 586CBEA4
 P 4250 7350
-F 0 "#PWR0122" H 4250 7100 50  0001 C CNN
+F 0 "#PWR121" H 4250 7100 50  0001 C CNN
 F 1 "GND" H 4250 7200 50  0000 C CNN
 F 2 "" H 4250 7350 50  0000 C CNN
@@
 Connection ~ 7750 2350
 $Comp
-L GND #PWR0123
+L GND #PWR125
 U 1 1 586B5B63
 P 7600 2750
-F 0 "#PWR0123" H 7600 2500 50  0001 C CNN
+F 0 "#PWR125" H 7600 2500 50  0001 C CNN
 F 1 "GND" H 7600 2600 50  0000 C CNN
 F 2 "" H 7600 2750 50  0000 C CNN
@@
 	4350 2350 5350 2350
 $Comp
-L +3.3V #PWR0124
+L +3.3V #PWR119
 U 1 1 58702007
 P 2950 2100
-F 0 "#PWR0124" H 2950 1950 50  0001 C CNN
+F 0 "#PWR119" H 2950 1950 50  0001 C CNN
 F 1 "+3.3V" H 2950 2240 50  0000 C CNN
 F 2 "" H 2950 2100 50  0000 C CNN
@@
 $EndComp
 $Comp
-L +5V #PWR0125
+L +5V #PWR128
 U 1 1 58716CC2
 P 8850 2150
-F 0 "#PWR0125" H 8850 2000 50  0001 C CNN
+F 0 "#PWR128" H 8850 2000 50  0001 C CNN
 F 1 "+5V" H 8850 2290 50  0000 C CNN
 F 2 "" H 8850 2150 50  0000 C CNN
@@
 $EndComp
 $Comp
-L +3.3V #PWR0126
+L +3.3V #PWR123
 U 1 1 58718360
 P 5000 6750
-F 0 "#PWR0126" H 5000 6600 50  0001 C CNN
+F 0 "#PWR123" H 5000 6600 50  0001 C CNN
 F 1 "+3.3V" H 5000 6890 50  0000 C CNN
 F 2 "" H 5000 6750 50  0000 C CNN
@@
 	7450 5150 7450 5300
 $Comp
-L GND #PWR0127
+L GND #PWR124
 U 1 1 587401D8
 P 7450 5300
-F 0 "#PWR0127" H 7450 5050 50  0001 C CNN
+F 0 "#PWR124" H 7450 5050 50  0001 C CNN
 F 1 "GND" H 7450 5150 50  0000 C CNN
 F 2 "" H 7450 5300 50  0000 C CNN
@@
 	5350 4250 4100 4250
 $Comp
-L +3.3V #PWR0128
+L +3.3V #PWR126
 U 1 1 5874294E
 P 8050 4600
-F 0 "#PWR0128" H 8050 4450 50  0001 C CNN
+F 0 "#PWR126" H 8050 4450 50  0001 C CNN
 F 1 "+3.3V" H 8050 4740 50  0000 C CNN
 F 2 "" H 8050 4600 50  0000 C CNN
@@
 	3750 6850 3750 6950
 $Comp
-L +3.3V #PWR0129
+L +3.3V #PWR116
 U 1 1 58742DE4
 P 1550 900
-F 0 "#PWR0129" H 1550 750 50  0001 C CNN
+F 0 "#PWR116" H 1550 750 50  0001 C CNN
 F 1 "+3.3V" H 1550 1040 50  0000 C CNN
 F 2 "" H 1550 900 50  0000 C CNN

Commit message: a few more footprints
Parts:
- D6: footprint (none) -> Diodes_SMD:SOD-523
- F1: footprint (none) -> Capacitors_SMD:C_1206
Changed lines of the file:
@@
 	1950 4050 3950 4050
 $Comp
-L GND #PWR120
+L GND #PWR0117
 U 1 1 58643EDD
 P 2950 6900
-F 0 "#PWR120" H 2950 6650 50  0001 C CNN
+F 0 "#PWR0117" H 2950 6650 50  0001 C CNN
 F 1 "GND" H 2950 6750 50  0000 C CNN
 F 2 "" H 2950 6900 50  0000 C CNN
@@
 Connection ~ 2150 6300
 $Comp
-L GND #PWR118
+L GND #PWR0118
 U 1 1 58644254
 P 2300 5300
-F 0 "#PWR118" H 2300 5050 50  0001 C CNN
+F 0 "#PWR0118" H 2300 5050 50  0001 C CNN
 F 1 "GND" H 2300 5150 50  0000 C CNN
 F 2 "" H 2300 5300 50  0000 C CNN
@@
 $EndComp
 $Comp
-L GND #PWR117
+L GND #PWR0119
 U 1 1 58644E40
 P 1800 2450
-F 0 "#PWR117" H 1800 2200 50  0001 C CNN
+F 0 "#PWR0119" H 1800 2200 50  0001 C CNN
 F 1 "GND" H 1800 2300 50  0000 C CNN
 F 2 "" H 1800 2450 50  0000 C CNN
@@
 F 0 "F1" H 10000 3150 60  0000 C CNN
 F 1 "PTS120630V012" H 10050 2950 60  0000 C CNN
-F 2 "" H 10000 3000 60  0001 C CNN
+F 2 "Capacitors_SMD:C_1206" H 10000 3000 60  0001 C CNN
 F 3 "" H 10000 3000 60  0001 C CNN
 	1    10050 3000
@@
 Connection ~ 8800 3700
 $Comp
-L GND #PWR127
+L GND #PWR0120
 U 1 1 586484F8
 P 8800 3850
-F 0 "#PWR127" H 8800 3600 50  0001 C CNN
+F 0 "#PWR0120" H 8800 3600 50  0001 C CNN
 F 1 "GND" H 8800 3700 50  0000 C CNN
 F 2 "" H 8800 3850 50  0000 C CNN
@@
 F 0 "D6" H 2950 2900 40  0000 C CNN
 F 1 "BAS16XV2T1G" H 2950 2700 40  0000 C CNN
-F 2 "" H 2950 2800 60  0001 C CNN
+F 2 "Diodes_SMD:SOD-523" H 2950 2800 60  0001 C CNN
 F 3 "" H 2950 2800 60  0000 C CNN
 	1    2950 2800
@@
 Connection ~ 3350 5650
 $Comp
-L GND #PWR122
+L GND #PWR0121
 U 1 1 58662B25
 P 4450 5300
-F 0 "#PWR122" H 4450 5050 50  0001 C CNN
+F 0 "#PWR0121" H 4450 5050 50  0001 C CNN
 F 1 "GND" H 4450 5150 50  0000 C CNN
 F 2 "" H 4450 5300 50  0000 C CNN
@@
 Connection ~ 4750 7250
 $Comp
-L GND #PWR121
+L GND #PWR0122
 U 1 1 586CBEA4
 P 4250 7350
-F 0 "#PWR121" H 4250 7100 50  0001 C CNN
+F 0 "#PWR0122" H 4250 7100 50  0001 C CNN
 F 1 "GND" H 4250 7200 50  0000 C CNN
 F 2 "" H 4250 7350 50  0000 C CNN
@@
 Connection ~ 7750 2350
 $Comp
-L GND #PWR125
+L GND #PWR0123
 U 1 1 586B5B63
 P 7600 2750
-F 0 "#PWR125" H 7600 2500 50  0001 C CNN
+F 0 "#PWR0123" H 7600 2500 50  0001 C CNN
 F 1 "GND" H 7600 2600 50  0000 C CNN
 F 2 "" H 7600 2750 50  0000 C CNN
@@
 	4350 2350 5350 2350
 $Comp
-L +3.3V #PWR119
+L +3.3V #PWR0124
 U 1 1 58702007
 P 2950 2100
-F 0 "#PWR119" H 2950 1950 50  0001 C CNN
+F 0 "#PWR0124" H 2950 1950 50  0001 C CNN
 F 1 "+3.3V" H 2950 2240 50  0000 C CNN
 F 2 "" H 2950 2100 50  0000 C CNN
@@
 $EndComp
 $Comp
-L +5V #PWR128
+L +5V #PWR0125
 U 1 1 58716CC2
 P 8850 2150
-F 0 "#PWR128" H 8850 2000 50  0001 C CNN
+F 0 "#PWR0125" H 8850 2000 50  0001 C CNN
 F 1 "+5V" H 8850 2290 50  0000 C CNN
 F 2 "" H 8850 2150 50  0000 C CNN
@@
 $EndComp
 $Comp
-L +3.3V #PWR123
+L +3.3V #PWR0126
 U 1 1 58718360
 P 5000 6750
-F 0 "#PWR123" H 5000 6600 50  0001 C CNN
+F 0 "#PWR0126" H 5000 6600 50  0001 C CNN
 F 1 "+3.3V" H 5000 6890 50  0000 C CNN
 F 2 "" H 5000 6750 50  0000 C CNN
@@
 	7450 5150 7450 5300
 $Comp
-L GND #PWR124
+L GND #PWR0127
 U 1 1 587401D8
 P 7450 5300
-F 0 "#PWR124" H 7450 5050 50  0001 C CNN
+F 0 "#PWR0127" H 7450 5050 50  0001 C CNN
 F 1 "GND" H 7450 5150 50  0000 C CNN
 F 2 "" H 7450 5300 50  0000 C CNN
@@
 	5350 4250 4100 4250
 $Comp
-L +3.3V #PWR126
+L +3.3V #PWR0128
 U 1 1 5874294E
 P 8050 4600
-F 0 "#PWR126" H 8050 4450 50  0001 C CNN
+F 0 "#PWR0128" H 8050 4450 50  0001 C CNN
 F 1 "+3.3V" H 8050 4740 50  0000 C CNN
 F 2 "" H 8050 4600 50  0000 C CNN
@@
 	3750 6850 3750 6950
 $Comp
-L +3.3V #PWR116
+L +3.3V #PWR0129
 U 1 1 58742DE4
 P 1550 900
-F 0 "#PWR116" H 1550 750 50  0001 C CNN
+F 0 "#PWR0129" H 1550 750 50  0001 C CNN
 F 1 "+3.3V" H 1550 1040 50  0000 C CNN
 F 2 "" H 1550 900 50  0000 C CNN

Commit message: A few more footprints
Parts:
- U1: footprint (none) -> SMD_Packages:BGA-256
Changed lines of the file:
@@
 F 0 "U1" H 5550 2100 60  0000 L CNN
 F 1 "xc7a50tftg256" H 5550 2000 60  0000 L CNN
-F 2 "" H 5350 1850 60  0001 C CNN
+F 2 "SMD_Packages:BGA-256" H 5350 1850 60  0001 C CNN
 F 3 "" H 5350 1850 60  0001 C CNN
 	5    5350 1850

Commit message: forgot to save sch
Parts:
- U11: footprint (none) -> so8:SO-8
- U12: footprint (none) -> TO_SOT_Packages_SMD:SC-70
- U13: footprint (none) -> TO_SOT_Packages_SMD:SOT-23
- U14: footprint (none) -> csp:WLCSP4_P0.5mm
Changed lines of the file:
@@
 F 0 "U11" H 2750 1500 60  0000 C CNN
 F 1 "GTL2002" H 2750 1300 60  0000 C CNN
-F 2 "" H 2750 1500 50  0001 C CNN
+F 2 "so8:SO-8" H 2750 1500 50  0001 C CNN
 F 3 "" H 2750 1500 60  0001 C CNN
 F 4 "568-4224-5-ND" H 2750 1500 50  0001 C CNN "Part Number"
@@
 F 0 "U14" H 9200 3500 60  0000 C CNN
 F 1 "ADP198ACPZ-R7" H 9500 3400 60  0000 C CNN
-F 2 "" H 8850 3000 60  0001 C CNN
+F 2 "csp:WLCSP4_P0.5mm" H 8850 3000 60  0001 C CNN
 F 3 "" H 8850 3000 60  0001 C CNN
 	1    8850 3000
@@
 F 0 "U12" H 2950 4750 60  0000 C CNN
 F 1 "NC7WZ07P6X" H 3500 4700 60  0000 C CNN
-F 2 "" H 3150 4850 60  0001 C CNN
+F 2 "TO_SOT_Packages_SMD:SC-70" H 3150 4850 60  0001 C CNN
 F 3 "" H 3150 4850 60  0001 C CNN
 	1    3150 4850
@@
 F 0 "U13" H 3000 5050 60  0000 C CNN
 F 1 "NC7SZ125M5X" H 3750 5000 60  0000 C CNN
-F 2 "" H 3330 5240 60  0001 C CNN
+F 2 "TO_SOT_Packages_SMD:SOT-23" H 3330 5240 60  0001 C CNN
 F 3 "" H 3330 5240 60  0001 C CNN
 	1    3250 5250

Commit message: new annotation
Parts:
- U1: footprint SMD_Packages:BGA-256 -> (none)
Changed lines of the file:
@@
 F 0 "U1" H 5550 2100 60  0000 L CNN
 F 1 "xc7a50tftg256" H 5550 2000 60  0000 L CNN
-F 2 "SMD_Packages:BGA-256" H 5350 1850 60  0001 C CNN
+F 2 "" H 5350 1850 60  0001 C CNN
 F 3 "" H 5350 1850 60  0001 C CNN
 	5    5350 1850
@@
 	1950 4050 3950 4050
 $Comp
-L GND #PWR0117
+L GND #PWR121
 U 1 1 58643EDD
 P 2950 6900
-F 0 "#PWR0117" H 2950 6650 50  0001 C CNN
+F 0 "#PWR121" H 2950 6650 50  0001 C CNN
 F 1 "GND" H 2950 6750 50  0000 C CNN
 F 2 "" H 2950 6900 50  0000 C CNN
@@
 Connection ~ 2150 6300
 $Comp
-L GND #PWR0118
+L GND #PWR119
 U 1 1 58644254
 P 2300 5300
-F 0 "#PWR0118" H 2300 5050 50  0001 C CNN
+F 0 "#PWR119" H 2300 5050 50  0001 C CNN
 F 1 "GND" H 2300 5150 50  0000 C CNN
 F 2 "" H 2300 5300 50  0000 C CNN
@@
 $EndComp
 $Comp
-L GND #PWR0119
+L GND #PWR118
 U 1 1 58644E40
 P 1800 2450
-F 0 "#PWR0119" H 1800 2200 50  0001 C CNN
+F 0 "#PWR118" H 1800 2200 50  0001 C CNN
 F 1 "GND" H 1800 2300 50  0000 C CNN
 F 2 "" H 1800 2450 50  0000 C CNN
@@
 Connection ~ 8800 3700
 $Comp
-L GND #PWR0120
+L GND #PWR128
 U 1 1 586484F8
 P 8800 3850
-F 0 "#PWR0120" H 8800 3600 50  0001 C CNN
+F 0 "#PWR128" H 8800 3600 50  0001 C CNN
 F 1 "GND" H 8800 3700 50  0000 C CNN
 F 2 "" H 8800 3850 50  0000 C CNN
@@
 Connection ~ 3350 5650
 $Comp
-L GND #PWR0121
+L GND #PWR123
 U 1 1 58662B25
 P 4450 5300
-F 0 "#PWR0121" H 4450 5050 50  0001 C CNN
+F 0 "#PWR123" H 4450 5050 50  0001 C CNN
 F 1 "GND" H 4450 5150 50  0000 C CNN
 F 2 "" H 4450 5300 50  0000 C CNN
@@
 Connection ~ 4750 7250
 $Comp
-L GND #PWR0122
+L GND #PWR122
 U 1 1 586CBEA4
 P 4250 7350
-F 0 "#PWR0122" H 4250 7100 50  0001 C CNN
+F 0 "#PWR122" H 4250 7100 50  0001 C CNN
 F 1 "GND" H 4250 7200 50  0000 C CNN
 F 2 "" H 4250 7350 50  0000 C CNN
@@
 Connection ~ 7750 2350
 $Comp
-L GND #PWR0123
+L GND #PWR126
 U 1 1 586B5B63
 P 7600 2750
-F 0 "#PWR0123" H 7600 2500 50  0001 C CNN
+F 0 "#PWR126" H 7600 2500 50  0001 C CNN
 F 1 "GND" H 7600 2600 50  0000 C CNN
 F 2 "" H 7600 2750 50  0000 C CNN
@@
 	4350 2350 5350 2350
 $Comp
-L +3.3V #PWR0124
+L +3.3V #PWR120
 U 1 1 58702007
 P 2950 2100
-F 0 "#PWR0124" H 2950 1950 50  0001 C CNN
+F 0 "#PWR120" H 2950 1950 50  0001 C CNN
 F 1 "+3.3V" H 2950 2240 50  0000 C CNN
 F 2 "" H 2950 2100 50  0000 C CNN
@@
 $EndComp
 $Comp
-L +5V #PWR0125
+L +5V #PWR129
 U 1 1 58716CC2
 P 8850 2150
-F 0 "#PWR0125" H 8850 2000 50  0001 C CNN
+F 0 "#PWR129" H 8850 2000 50  0001 C CNN
 F 1 "+5V" H 8850 2290 50  0000 C CNN
 F 2 "" H 8850 2150 50  0000 C CNN
@@
 $EndComp
 $Comp
-L +3.3V #PWR0126
+L +3.3V #PWR124
 U 1 1 58718360
 P 5000 6750
-F 0 "#PWR0126" H 5000 6600 50  0001 C CNN
+F 0 "#PWR124" H 5000 6600 50  0001 C CNN
 F 1 "+3.3V" H 5000 6890 50  0000 C CNN
 F 2 "" H 5000 6750 50  0000 C CNN
@@
 	7450 5150 7450 5300
 $Comp
-L GND #PWR0127
+L GND #PWR125
 U 1 1 587401D8
 P 7450 5300
-F 0 "#PWR0127" H 7450 5050 50  0001 C CNN
+F 0 "#PWR125" H 7450 5050 50  0001 C CNN
 F 1 "GND" H 7450 5150 50  0000 C CNN
 F 2 "" H 7450 5300 50  0000 C CNN
@@
 	5350 4250 4100 4250
 $Comp
-L +3.3V #PWR0128
+L +3.3V #PWR127
 U 1 1 5874294E
 P 8050 4600
-F 0 "#PWR0128" H 8050 4450 50  0001 C CNN
+F 0 "#PWR127" H 8050 4450 50  0001 C CNN
 F 1 "+3.3V" H 8050 4740 50  0000 C CNN
 F 2 "" H 8050 4600 50  0000 C CNN
@@
 	3750 6850 3750 6950
 $Comp
-L +3.3V #PWR0129
+L +3.3V #PWR117
 U 1 1 58742DE4
 P 1550 900
-F 0 "#PWR0129" H 1550 750 50  0001 C CNN
+F 0 "#PWR117" H 1550 750 50  0001 C CNN
 F 1 "+3.3V" H 1550 1040 50  0000 C CNN
 F 2 "" H 1550 900 50  0000 C CNN

Commit message: A few more footprints
Parts:
- U1: footprint (none) -> SMD_Packages:BGA-256
Changed lines of the file:
@@
 F 0 "U1" H 5550 2100 60  0000 L CNN
 F 1 "xc7a50tftg256" H 5550 2000 60  0000 L CNN
-F 2 "" H 5350 1850 60  0001 C CNN
+F 2 "SMD_Packages:BGA-256" H 5350 1850 60  0001 C CNN
 F 3 "" H 5350 1850 60  0001 C CNN
 	5    5350 1850
@@
 	1950 4050 3950 4050
 $Comp
-L GND #PWR121
+L GND #PWR0118
 U 1 1 58643EDD
 P 2950 6900
-F 0 "#PWR121" H 2950 6650 50  0001 C CNN
+F 0 "#PWR0118" H 2950 6650 50  0001 C CNN
 F 1 "GND" H 2950 6750 50  0000 C CNN
 F 2 "" H 2950 6900 50  0000 C CNN
@@
 Connection ~ 2150 6300
 $Comp
-L GND #PWR119
+L GND #PWR0119
 U 1 1 58644254
 P 2300 5300
-F 0 "#PWR119" H 2300 5050 50  0001 C CNN
+F 0 "#PWR0119" H 2300 5050 50  0001 C CNN
 F 1 "GND" H 2300 5150 50  0000 C CNN
 F 2 "" H 2300 5300 50  0000 C CNN
@@
 $EndComp
 $Comp
-L GND #PWR118
+L GND #PWR0120
 U 1 1 58644E40
 P 1800 2450
-F 0 "#PWR118" H 1800 2200 50  0001 C CNN
+F 0 "#PWR0120" H 1800 2200 50  0001 C CNN
 F 1 "GND" H 1800 2300 50  0000 C CNN
 F 2 "" H 1800 2450 50  0000 C CNN
@@
 Connection ~ 8800 3700
 $Comp
-L GND #PWR128
+L GND #PWR0121
 U 1 1 586484F8
 P 8800 3850
-F 0 "#PWR128" H 8800 3600 50  0001 C CNN
+F 0 "#PWR0121" H 8800 3600 50  0001 C CNN
 F 1 "GND" H 8800 3700 50  0000 C CNN
 F 2 "" H 8800 3850 50  0000 C CNN
@@
 Connection ~ 3350 5650
 $Comp
-L GND #PWR123
+L GND #PWR0122
 U 1 1 58662B25
 P 4450 5300
-F 0 "#PWR123" H 4450 5050 50  0001 C CNN
+F 0 "#PWR0122" H 4450 5050 50  0001 C CNN
 F 1 "GND" H 4450 5150 50  0000 C CNN
 F 2 "" H 4450 5300 50  0000 C CNN
@@
 Connection ~ 4750 7250
 $Comp
-L GND #PWR122
+L GND #PWR0123
 U 1 1 586CBEA4
 P 4250 7350
-F 0 "#PWR122" H 4250 7100 50  0001 C CNN
+F 0 "#PWR0123" H 4250 7100 50  0001 C CNN
 F 1 "GND" H 4250 7200 50  0000 C CNN
 F 2 "" H 4250 7350 50  0000 C CNN
@@
 Connection ~ 7750 2350
 $Comp
-L GND #PWR126
+L GND #PWR0124
 U 1 1 586B5B63
 P 7600 2750
-F 0 "#PWR126" H 7600 2500 50  0001 C CNN
+F 0 "#PWR0124" H 7600 2500 50  0001 C CNN
 F 1 "GND" H 7600 2600 50  0000 C CNN
 F 2 "" H 7600 2750 50  0000 C CNN
@@
 	4350 2350 5350 2350
 $Comp
-L +3.3V #PWR120
+L +3.3V #PWR0125
 U 1 1 58702007
 P 2950 2100
-F 0 "#PWR120" H 2950 1950 50  0001 C CNN
+F 0 "#PWR0125" H 2950 1950 50  0001 C CNN
 F 1 "+3.3V" H 2950 2240 50  0000 C CNN
 F 2 "" H 2950 2100 50  0000 C CNN
@@
 $EndComp
 $Comp
-L +5V #PWR129
+L +5V #PWR0126
 U 1 1 58716CC2
 P 8850 2150
-F 0 "#PWR129" H 8850 2000 50  0001 C CNN
+F 0 "#PWR0126" H 8850 2000 50  0001 C CNN
 F 1 "+5V" H 8850 2290 50  0000 C CNN
 F 2 "" H 8850 2150 50  0000 C CNN
@@
 $EndComp
 $Comp
-L +3.3V #PWR124
+L +3.3V #PWR0127
 U 1 1 58718360
 P 5000 6750
-F 0 "#PWR124" H 5000 6600 50  0001 C CNN
+F 0 "#PWR0127" H 5000 6600 50  0001 C CNN
 F 1 "+3.3V" H 5000 6890 50  0000 C CNN
 F 2 "" H 5000 6750 50  0000 C CNN
@@
 	7450 5150 7450 5300
 $Comp
-L GND #PWR125
+L GND #PWR0128
 U 1 1 587401D8
 P 7450 5300
-F 0 "#PWR125" H 7450 5050 50  0001 C CNN
+F 0 "#PWR0128" H 7450 5050 50  0001 C CNN
 F 1 "GND" H 7450 5150 50  0000 C CNN
 F 2 "" H 7450 5300 50  0000 C CNN
@@
 	5350 4250 4100 4250
 $Comp
-L +3.3V #PWR127
+L +3.3V #PWR0129
 U 1 1 5874294E
 P 8050 4600
-F 0 "#PWR127" H 8050 4450 50  0001 C CNN
+F 0 "#PWR0129" H 8050 4450 50  0001 C CNN
 F 1 "+3.3V" H 8050 4740 50  0000 C CNN
 F 2 "" H 8050 4600 50  0000 C CNN
@@
 	3750 6850 3750 6950
 $Comp
-L +3.3V #PWR117
+L +3.3V #PWR0130
 U 1 1 58742DE4
 P 1550 900
-F 0 "#PWR117" H 1550 750 50  0001 C CNN
+F 0 "#PWR0130" H 1550 750 50  0001 C CNN
 F 1 "+3.3V" H 1550 1040 50  0000 C CNN
 F 2 "" H 1550 900 50  0000 C CNN
