File: Memory.sch (KiCad schematic (older format))
At the start: 8 parts, among them U2 24FC128, U3 N25Q128A

Commit message: added resistor footprints (1206)
Parts:
- R75, R82: footprint (none) -> Resistors_SMD:R_1206
Changed lines of the file:
@@
 F 0 "R75" H 6980 4320 50  0000 L CNN
 F 1 "20k" H 6980 4260 50  0000 L CNN
-F 2 "" H 6950 4300 50  0001 C CNN
+F 2 "Resistors_SMD:R_1206" H 6950 4300 50  0001 C CNN
 F 3 "" H 6950 4300 50  0000 C CNN
 	1    6950 4300
@@
 F 0 "R82" H 4830 3720 50  0000 L CNN
 F 1 "50k" H 4830 3660 50  0000 L CNN
-F 2 "" H 4800 3700 50  0001 C CNN
+F 2 "Resistors_SMD:R_1206" H 4800 3700 50  0001 C CNN
 F 3 "" H 4800 3700 50  0000 C CNN
 	1    4800 3700

Commit message: ???
Parts:
- U3: footprint (none) -> VPDFN8:V-PDFN-8 6mmx5mm Sawm (MLP8)
Changed lines of the file:
@@
 I2C_SDIN
 $Comp
-L +1.8V #PWR47
+L +1.8V #PWR045
 U 1 1 58594FA1
 P 5450 1100
-F 0 "#PWR47" H 5450 1240 20  0001 C CNN
+F 0 "#PWR045" H 5450 1240 20  0001 C CNN
 F 1 "+1.8V" H 5450 1210 30  0000 C CNN
 F 2 "" H 5450 1100 60  0001 C CNN
@@
 $EndComp
 $Comp
-L GND-RESCUE-DFTBoard #PWR45
+L GND-RESCUE-DFTBoard #PWR046
 U 1 1 58594FE3
 P 4600 1950
-F 0 "#PWR45" H 4600 1950 30  0001 C CNN
+F 0 "#PWR046" H 4600 1950 30  0001 C CNN
 F 1 "GND" H 4600 1880 30  0001 C CNN
 F 2 "" H 4600 1950 60  0001 C CNN
@@
 $EndComp
 $Comp
-L GND-RESCUE-DFTBoard #PWR48
+L GND-RESCUE-DFTBoard #PWR047
 U 1 1 58594FFB
 P 5450 2350
-F 0 "#PWR48" H 5450 2350 30  0001 C CNN
+F 0 "#PWR047" H 5450 2350 30  0001 C CNN
 F 1 "GND" H 5450 2280 30  0001 C CNN
 F 2 "" H 5450 2350 60  0001 C CNN
@@
 F 0 "U3" H 5700 3950 50  0000 C CNN
 F 1 "N25Q128A" H 5900 3450 50  0000 C CNN
-F 2 "" H 5700 4050 50  0001 C CNN
+F 2 "VPDFN8:V-PDFN-8 6mmx5mm Sawm (MLP8)" H 5700 4050 50  0001 C CNN
 F 3 "DOCUMENTATION" H 5700 4050 50  0001 C CNN
 	1    5700 4050
@@
 	6650 4300 6650 4750
 $Comp
-L GND #PWR50
+L GND #PWR048
 U 1 1 58666BA4
 P 6650 4750
-F 0 "#PWR50" H 6650 4500 50  0001 C CNN
+F 0 "#PWR048" H 6650 4500 50  0001 C CNN
 F 1 "GND" H 6650 4600 50  0000 C CNN
 F 2 "" H 6650 4750 50  0000 C CNN
@@
 	4350 4400 4950 4400
 $Comp
-L +1.8V #PWR46
+L +1.8V #PWR049
 U 1 1 5868C7CB
 P 4600 3500
-F 0 "#PWR46" H 4600 3640 20  0001 C CNN
+F 0 "#PWR049" H 4600 3640 20  0001 C CNN
 F 1 "+1.8V" H 4600 3610 30  0000 C CNN
 F 2 "" H 4600 3500 60  0001 C CNN
@@
 	6450 4400 6950 4400
 $Comp
-L +1.8V #PWR51
+L +1.8V #PWR050
 U 1 1 5868C8FE
 P 6950 4150
-F 0 "#PWR51" H 6950 4290 20  0001 C CNN
+F 0 "#PWR050" H 6950 4290 20  0001 C CNN
 F 1 "+1.8V" H 6950 4260 30  0000 C CNN
 F 2 "" H 6950 4150 60  0001 C CNN
@@
 Connection ~ 5800 1150
 $Comp
-L GND-RESCUE-DFTBoard #PWR49
+L GND-RESCUE-DFTBoard #PWR051
 U 1 1 586C114A
 P 6000 1500
-F 0 "#PWR49" H 6000 1500 30  0001 C CNN
+F 0 "#PWR051" H 6000 1500 30  0001 C CNN
 F 1 "GND" H 6000 1430 30  0001 C CNN
 F 2 "" H 6000 1500 60  0001 C CNN
@@
 $EndComp
 $Comp
-L GND-RESCUE-DFTBoard #PWR44
+L GND-RESCUE-DFTBoard #PWR052
 U 1 1 586C1999
 P 4250 4050
-F 0 "#PWR44" H 4250 4050 30  0001 C CNN
+F 0 "#PWR052" H 4250 4050 30  0001 C CNN
 F 1 "GND" H 4250 3980 30  0001 C CNN
 F 2 "" H 4250 4050 60  0001 C CNN

Commit message: fixed a few diagram/footprint pin mismatches, getting ready to pull gene's microhdmi footprint
Parts:
- U3: footprint VPDFN8:V-PDFN-8 6mmx5mm Sawm (MLP8) -> DFTcustom:V-PDFN-8 6mmx5mm Sawm (MLP8)
Changed lines of the file:
@@
 LIBS:ferrite
 LIBS:df_device
+LIBS:JACK_TRS_5PINS
 EELAYER 25 0
 EELAYER END
@@
 F 0 "U3" H 5700 3950 50  0000 C CNN
 F 1 "N25Q128A" H 5900 3450 50  0000 C CNN
-F 2 "VPDFN8:V-PDFN-8 6mmx5mm Sawm (MLP8)" H 5700 4050 50  0001 C CNN
+F 2 "DFTcustom:V-PDFN-8 6mmx5mm Sawm (MLP8)" H 5700 4050 50  0001 C CNN
 F 3 "DOCUMENTATION" H 5700 4050 50  0001 C CNN
 	1    5700 4050

Commit message: a few small changes
Parts:
- U3: footprint DFTcustom:V-PDFN-8 6mmx5mm Sawm (MLP8) -> SMD_Packages:SO-16-N
Changed lines of the file:
@@
 F 0 "U3" H 5700 3950 50  0000 C CNN
 F 1 "N25Q128A" H 5900 3450 50  0000 C CNN
-F 2 "DFTcustom:V-PDFN-8 6mmx5mm Sawm (MLP8)" H 5700 4050 50  0001 C CNN
+F 2 "SMD_Packages:SO-16-N" H 5700 4050 50  0001 C CNN
 F 3 "DOCUMENTATION" H 5700 4050 50  0001 C CNN
 	1    5700 4050
