File: DFTBoard.kicad_pcb (KiCad board)
At the start: 10 copper layers, 265 x 60 mm, 315 parts, among them CON1 AVR-JTAG-10, CON2 AVR-JTAG-10, IC1 WM8758B, IC2 IS31FL3199, IC3 CyUSB30xx-BZX, J1 JACK_TRS_5PINS, J2 JACK_TRS_5PINS, J3 JACK_TRS_5PINS, J4 JACK_TRS_5PINS, J5 GSB3211311WEU, J6 48258-0001, J7 MICRO_HDMI, J8 GSB3211311WEU, J9 48258-0001, Q1 IRLML2502, Q2 IRLML2502, Q3 IRLML2502, Q4 IRLML2502, Q5 IRLML2502, Q6 IRLML2502, SW1 SW_IL, U1 xc7a50tftg256, U10 NC7WZ07P6X, U11 NC7SZ125M5X, U12 GTL2002, U13 ADP198ACPZ-R7, U14 W9751G6KB, U15 CY7C65634-28LTXC, U2 24FC128, U3 W25Q128FW, U4 SC189 - 3.3V, U5 SC189 - 1.0V, U6 SC189 - 1.2V, U7 SC189 - 1.8V, U8 VL53L0X, U9 MAX3421, X1 KC5032A, Y1 19.2MHz, Y2 ECS-120-20-3X-TR, Y3 ECS-120-20-3X-TR

Commit message: finished wiring GPIF with exception of PCLK
Parts:
- removed ROT3: ROTARY-ENCODER, DFTcustom:rightangleencoders
- added ROT0: ROTARY-ENCODER, DFTcustom:rightangleencoders, F.Cu at (188.6, 100.2)
- C127, C128, C130, C131, C132, C133, C138, C141, C142, FB2, GT1, J7, R10, R12, R13, R16, R18, R21, R24, R26, R27, R29, R30, R56, R57, R8, R9: moved to B.Cu
- moved R94 240.9 mm to (260.3, 102.4), turned to 180 degrees
- moved C126 216.8 mm to (230.2, 120.0)
- moved C133 207.4 mm to (226.4, 115.6), turned to 90 degrees
- moved C129 204.2 mm to (227.5, 122.8), turned to 90 degrees
- moved C128 203.9 mm to (221.4, 115.6), turned to 90 degrees
- moved C127 203.9 mm to (221.4, 119.6), turned to 90 degrees
- moved C132 197.8 mm to (226.4, 119.6), turned to 90 degrees
- moved C130 190.1 mm to (214.3, 115.6), turned to 270 degrees
- moved C131 185.5 mm to (214.3, 112.4), turned to 270 degrees
- moved R44 157.5 mm to (239.2, 115.2), turned to 180 degrees
- moved R27 146.5 mm to (211.7, 137.6)
- moved J6 132.5 mm to (273.1, 123.0), turned to 90 degrees
- moved CON1 127.0 mm to (210.6, 157.5), turned to 90 degrees
- moved R92 115.5 mm to (255.7, 102.4), turned to 180 degrees
- moved C36 113.1 mm to (64.5, 128.6), turned to 90 degrees
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Connections:
- net Net-(C127-Pad2) renamed /RAM/VREF
- net Net-(IC3-PadE10) renamed /Cypress FX3/VBATT
- net Net-(R44-Pad2) renamed /Memory/SPIMEM_WP
- net Net-(R45-Pad2) renamed /Memory/SPIMEM_RST
- net Net-(R82-Pad2) renamed /Encoders/ROT2A
- net Net-(R84-Pad2) renamed /Encoders/ROT2B
- net Net-(R92-Pad2) renamed /Encoders/ROT3A
- net Net-(R94-Pad2) renamed /Encoders/ROT3B
- R81 pad 2: Net-(R81-Pad2) -> /Encoders/ROT0A
- R83 pad 2: Net-(R83-Pad2) -> /Encoders/ROT0B
- R85 pad 2: Net-(R81-Pad2) -> /Encoders/ROT0A
- R86 pad 2: Net-(R83-Pad2) -> /Encoders/ROT0B
- R91 pad 2: Net-(R91-Pad2) -> /Encoders/ROT1A
- R93 pad 2: Net-(R93-Pad2) -> /Encoders/ROT1B
- R95 pad 2: Net-(R91-Pad2) -> /Encoders/ROT1A
- R96 pad 2: Net-(R93-Pad2) -> /Encoders/ROT1B
- ROT1 pad A: Net-(R81-Pad2) -> /Encoders/ROT1A
- ROT1 pad B: Net-(R83-Pad2) -> /Encoders/ROT1B
- ROT1 pad S1: ENCC0_SW -> ENCC1_SW
- U1 pad A10: RAM_LDM -> RAM_DQ12
- U1 pad A12: RAM_DQ2 -> RAM_LDQS_N
- U1 pad A13: RAM_DQ7 -> RAM_DQ0
- U1 pad A14: RAM_DQ6 -> RAM_DQ3
- U1 pad A15: RAM_DQ10 -> RAM_DQ5
- U1 pad A8: RAM_UDQS_P -> RAM_UDM
- U1 pad A9: RAM_UDQS_N -> RAM_DQ9
- U1 pad B10: RAM_DQ1 -> RAM_DQ13
- U1 pad B11: RAM_DQ0 -> RAM_LDM
- U1 pad B12: RAM_DQ3 -> RAM_LDQS_P
- U1 pad B14: RAM_DQ8 -> RAM_DQ4
- U1 pad B15: RAM_DQ11 -> RAM_DQ2
- U1 pad B16: RAM_DQ12 -> (no net)
- U1 pad B9: RAM_UDM -> RAM_DQ8
- U1 pad C11: RAM_DQ15 -> RAM_DQ6
- U1 pad C12: RAM_DQ14 -> RAM_DQ1
- U1 pad C14: RAM_DQ9 -> RAM_RAS#
- U1 pad C16: RAM_DQ13 -> (no net)
- U1 pad C4: CLK100MHz -> (no net)
- U1 pad C8: RAM_LDQS_P -> RAM_UDQS_P
- U1 pad C9: RAM_LDQS_N -> RAM_UDQS_N
- U1 pad D11: RAM_A2 -> RAM_DQ11
- U1 pad D14: RAM_A5 -> RAM_CKE
- U1 pad D15: RAM_A4 -> RAM_WE#
- U1 pad D16: RAM_A8 -> RAM_CAS#
- U1 pad D4: (no net) -> CLK100MHz
- U1 pad D8: RAM_DQ5 -> RAM_DQ14
- U1 pad D9: RAM_DQ4 -> RAM_DQ15
- U1 pad E11: RAM_A3 -> RAM_DQ10
- U1 pad E12: RAM_A1 -> RAM_DQ7
- U1 pad E13: RAM_A0 -> RAM_BA1
- U1 pad E15: RAM_A10 -> RAM_A1
- U1 pad E16: RAM_A9 -> RAM_A10
- U1 pad F13: RAM_A6 -> RAM_A5
- U1 pad F14: RAM_CS# -> RAM_BA0
- U1 pad F15: RAM_A11 -> RAM_A3
- U1 pad G12: RAM_A12 -> RAM_A9
- U1 pad G14: RAM_CKE -> RAM_A2
- U1 pad G15: RAM_RAS# -> RAM_CS#
- U1 pad G16: RAM_CK_N -> RAM_A12
- U1 pad H12: RAM_BA1 -> RAM_A6
- U1 pad H13: RAM_BA0 -> RAM_A11
- U1 pad H16: RAM_CK_P -> RAM_A0
- U1 pad J13: GPIF_FLAGAT -> GA_0T
- U1 pad J14: GPIF_FLAGBT -> GA_1T
- U1 pad J15: RAM_CAS# -> RAM_A8
- U1 pad J16: RAM_WE# -> RAM_A4
- U1 pad K12: GPIF_SLCS#T -> (no net)
- U1 pad K13: GD_10T -> GPIF_SLWR#T
- U1 pad K15: GD_13T -> GPIF_FLAGAT
- U1 pad K16: GD_11T -> GPIF_FLAGBT
- U1 pad L12: GA_0T -> GD_4T
- U1 pad L13: GD_8T -> GD_14T
- U1 pad L14: GD_9T -> GPIF_SLOE#T
- U1 pad L15: GD_14T -> GPIF_SLRD#T
- U1 pad M12: GD_6T -> GD_12T
- U1 pad M14: GD_7T -> GD_13T
- U1 pad M15: GD_12T -> GPIF_SLCS#T
- U1 pad M16: GA_1T -> GPIF_PKTEND#T
- U1 pad N11: (no net) -> GPIF_PCLKT
- U1 pad N12: I2S_BCLK -> I2S_MCLK
- U1 pad N13: GPIF_SLRD#T -> GD_11T
- U1 pad N14: I2S_MCLK -> I2S_BCLK
- U1 pad N16: GD_15T -> GD_9T
- U1 pad P11: (no net) -> GD_0T
- U1 pad P13: GPIF_PKTEND#T -> GD_15T
- U1 pad P15: GD_3T -> GD_8T
- U1 pad P16: GD_4T -> GD_10T
- U1 pad R11: (no net) -> GD_1T
- U1 pad R12: (no net) -> GD_2T
- U1 pad R15: GD_2T -> GD_7T
- U1 pad R16: GD_5T -> GD_6T
- U1 pad T10: GPIF_SLOE#T -> (no net)
- U1 pad T14: GD_0T -> GD_3T
- U1 pad T15: GD_1T -> GD_5T
- U1 pad T8: GPIF_SLWR#T -> (no net)
- U1 pad T9: GPIF_PCLKT -> (no net)
Routing:
- net /RAM/VREF: track 0.00 -> 22.4 mm, vias 0 -> 1
- net /Audio/HPLOUT: track 0.00 -> 21.6 mm
- net /Audio/HPROUT: track 0.00 -> 21.6 mm
- net GD_13: track 0.00 -> 21.4 mm, vias 0 -> 2
- net GD_2: track 8.06 -> 28.9 mm, vias 1 -> 2
- net GD_15: track 5.20 -> 25.2 mm, vias 1 -> 2
- net GPIF_SLOE#: track 0.00 -> 19.7 mm, vias 0 -> 2
- net GPIF_FLAGA: track 2.52 -> 21.5 mm, vias 1 -> 2
- net (no net): track 23.6 -> 4.71 mm, vias 0 -> 2
- net GPIF_SLCS#: track 0.00 -> 18.6 mm, vias 0 -> 2
- net GPIF_FLAGB: track 5.94 -> 24.0 mm, vias 1 -> 2
- net GD_4: track 4.40 -> 22.1 mm, vias 1 -> 2
- net TEMPO_SW: track 18.2 -> 0.82 mm, vias 0 -> 1
- net RAM_DQ12: track 33.9 -> 17.1 mm
- net GD_7: track 4.36 -> 21.1 mm, vias 1 -> 2
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- added copper zone on GND0, net GND
- removed copper zone on GND, net GND
