File: FPGA Unused IO.sch (KiCad schematic (older format))
At the start: 1 part, among them U1 xc7a50tftg256

Commit message: more moving around components and connecting. all cypress and FPGA bypass caps placed
Parts:
- removed unit 3 of U1
Connections:
- no-connect marks 70 -> 20
Changed lines of the file:
@@
 LIBS:gndtie
 LIBS:powerswitch
+LIBS:winbond
+LIBS:cy7c65634-28ltxc
+LIBS:powerjumper
 EELAYER 25 0
 EELAYER END
 $Descr A4 11693 8268
 encoding utf-8
-Sheet 6 15
+Sheet 6 16
 Title ""
 Date ""
@@
 Comment4 ""
 $EndDescr
-$Comp
-L xc7a50tftg256 U1
-U 3 1 585C5883
-P 1850 1450
-F 0 "U1" H 2050 1700 60  0000 L CNN
-F 1 "xc7a50tftg256" H 2050 1600 60  0000 L CNN
-F 2 "SMD_Packages:BGA-256" H 1850 1450 60  0001 C CNN
-F 3 "" H 1850 1450 60  0001 C CNN
-	3    1850 1450
-	1    0    0    -1
-$EndComp
 NoConn ~ 4950 2150
 NoConn ~ 4950 2250
@@
 NoConn ~ 4950 3750
 NoConn ~ 4950 3850
-NoConn ~ 1850 2450
-NoConn ~ 1850 2550
-NoConn ~ 1850 2650
-NoConn ~ 1850 2750
-NoConn ~ 1850 2850
-NoConn ~ 1850 2950
-NoConn ~ 1850 3050
-NoConn ~ 1850 3150
-NoConn ~ 1850 3250
-NoConn ~ 1850 3350
-NoConn ~ 1850 1450
-NoConn ~ 1850 1550
-NoConn ~ 1850 1650
-NoConn ~ 1850 1750
-NoConn ~ 1850 1850
-NoConn ~ 1850 1950
-NoConn ~ 1850 2050
-NoConn ~ 1850 2150
-NoConn ~ 1850 2250
-NoConn ~ 1850 2350
-NoConn ~ 1850 4450
-NoConn ~ 1850 4550
-NoConn ~ 1850 4650
-NoConn ~ 1850 4750
-NoConn ~ 1850 4850
-NoConn ~ 1850 4950
-NoConn ~ 1850 5050
-NoConn ~ 1850 5150
-NoConn ~ 1850 5250
-NoConn ~ 1850 5350
-NoConn ~ 1850 3450
-NoConn ~ 1850 3550
-NoConn ~ 1850 3650
-NoConn ~ 1850 3750
-NoConn ~ 1850 3850
-NoConn ~ 1850 3950
-NoConn ~ 1850 4050
-NoConn ~ 1850 4150
-NoConn ~ 1850 4250
-NoConn ~ 1850 4350
-NoConn ~ 1850 5450
-NoConn ~ 1850 5550
-NoConn ~ 1850 5650
-NoConn ~ 1850 5750
-NoConn ~ 1850 5850
-NoConn ~ 1850 5950
-NoConn ~ 1850 6050
-NoConn ~ 1850 6150
-NoConn ~ 1850 6250
-NoConn ~ 1850 6350
 $Comp
 L xc7a50tftg256 U1
@@
 $EndComp
 $Comp
-L GND #PWR25
-U 1 1 586E8826
-P 1650 6600
-F 0 "#PWR25" H 1650 6350 50  0001 C CNN
-F 1 "GND" H 1650 6450 50  0000 C CNN
-F 2 "" H 1650 6600 50  0000 C CNN
-F 3 "" H 1650 6600 50  0000 C CNN
-	1    1650 6600
-	1    0    0    -1
-$EndComp
-Wire Wire Line
-	1850 6450 1650 6450
-Wire Wire Line
-	1650 6450 1650 6600
-$Comp
-L GND #PWR26
+L GND #PWR025
 U 1 1 586E88A6
 P 4750 4300
-F 0 "#PWR26" H 4750 4050 50  0001 C CNN
+F 0 "#PWR025" H 4750 4050 50  0001 C CNN
 F 1 "GND" H 4750 4150 50  0000 C CNN
 F 2 "" H 4750 4300 50  0000 C CNN
