File: gpif2.sch (KiCad schematic (older format))
At the start: 38 parts, among them Q3 IRLML2502, SW1 TL6215RF200BDT, U1 xc7a50tftg256

Commit message: swapped 0201s for 0402 packages, currently reworking PDS so that 3.3V and 1.8V layers can be eliminated
Parts:
- R10, R11, R12, R13, R14, R15, R16, R17, R18, R19, R20, R21, R22, R23, R24, R25, R26, R27, R28, R29, R30, R31, R6, R7, R8, R9: footprint Resistors_SMD:R_0201 -> Resistors_SMD:R_0402
Changed lines of the file:
@@
 F 0 "R30" V 3880 1150 50  0000 C CNN
 F 1 "22" V 3800 1150 50  0000 C CNN
-F 2 "Resistors_SMD:R_0201" V 3730 1150 50  0001 C CNN
+F 2 "Resistors_SMD:R_0402" V 3730 1150 50  0001 C CNN
 F 3 "" H 3800 1150 50  0000 C CNN
 	1    3800 1150
@@
 F 0 "R23" V 3630 1250 50  0000 C CNN
 F 1 "22" V 3550 1250 50  0000 C CNN
-F 2 "Resistors_SMD:R_0201" V 3480 1250 50  0001 C CNN
+F 2 "Resistors_SMD:R_0402" V 3480 1250 50  0001 C CNN
 F 3 "" H 3550 1250 50  0000 C CNN
 	1    3550 1250
@@
 F 0 "R16" V 3380 1350 50  0000 C CNN
 F 1 "22" V 3300 1350 50  0000 C CNN
-F 2 "Resistors_SMD:R_0201" V 3230 1350 50  0001 C CNN
+F 2 "Resistors_SMD:R_0402" V 3230 1350 50  0001 C CNN
 F 3 "" H 3300 1350 50  0000 C CNN
 	1    3300 1350
@@
 F 0 "R10" V 3130 1450 50  0000 C CNN
 F 1 "22" V 3050 1450 50  0000 C CNN
-F 2 "Resistors_SMD:R_0201" V 2980 1450 50  0001 C CNN
+F 2 "Resistors_SMD:R_0402" V 2980 1450 50  0001 C CNN
 F 3 "" H 3050 1450 50  0000 C CNN
 	1    3050 1450
@@
 F 0 "R31" V 3880 1550 50  0000 C CNN
 F 1 "22" V 3800 1550 50  0000 C CNN
-F 2 "Resistors_SMD:R_0201" V 3730 1550 50  0001 C CNN
+F 2 "Resistors_SMD:R_0402" V 3730 1550 50  0001 C CNN
 F 3 "" H 3800 1550 50  0000 C CNN
 	1    3800 1550
@@
 F 0 "R24" V 3630 1650 50  0000 C CNN
 F 1 "22" V 3550 1650 50  0000 C CNN
-F 2 "Resistors_SMD:R_0201" V 3480 1650 50  0001 C CNN
+F 2 "Resistors_SMD:R_0402" V 3480 1650 50  0001 C CNN
 F 3 "" H 3550 1650 50  0000 C CNN
 	1    3550 1650
@@
 F 0 "R17" V 3380 1750 50  0000 C CNN
 F 1 "22" V 3300 1750 50  0000 C CNN
-F 2 "Resistors_SMD:R_0201" V 3230 1750 50  0001 C CNN
+F 2 "Resistors_SMD:R_0402" V 3230 1750 50  0001 C CNN
 F 3 "" H 3300 1750 50  0000 C CNN
 	1    3300 1750
@@
 F 0 "R11" V 3130 1850 50  0000 C CNN
 F 1 "22" V 3050 1850 50  0000 C CNN
-F 2 "Resistors_SMD:R_0201" V 2980 1850 50  0001 C CNN
+F 2 "Resistors_SMD:R_0402" V 2980 1850 50  0001 C CNN
 F 3 "" H 3050 1850 50  0000 C CNN
 	1    3050 1850
@@
 F 0 "R25" V 3780 2550 50  0000 C CNN
 F 1 "22" V 3700 2550 50  0000 C CNN
-F 2 "Resistors_SMD:R_0201" V 3630 2550 50  0001 C CNN
+F 2 "Resistors_SMD:R_0402" V 3630 2550 50  0001 C CNN
 F 3 "" H 3700 2550 50  0000 C CNN
 	1    3700 2550
@@
 F 0 "R18" V 3530 2650 50  0000 C CNN
 F 1 "22" V 3450 2650 50  0000 C CNN
-F 2 "Resistors_SMD:R_0201" V 3380 2650 50  0001 C CNN
+F 2 "Resistors_SMD:R_0402" V 3380 2650 50  0001 C CNN
 F 3 "" H 3450 2650 50  0000 C CNN
 	1    3450 2650
@@
 F 0 "R12" V 3280 2750 50  0000 C CNN
 F 1 "22" V 3200 2750 50  0000 C CNN
-F 2 "Resistors_SMD:R_0201" V 3130 2750 50  0001 C CNN
+F 2 "Resistors_SMD:R_0402" V 3130 2750 50  0001 C CNN
 F 3 "" H 3200 2750 50  0000 C CNN
 	1    3200 2750
@@
 F 0 "R6" V 3030 2850 50  0000 C CNN
 F 1 "22" V 2950 2850 50  0000 C CNN
-F 2 "Resistors_SMD:R_0201" V 2880 2850 50  0001 C CNN
+F 2 "Resistors_SMD:R_0402" V 2880 2850 50  0001 C CNN
 F 3 "" H 2950 2850 50  0000 C CNN
 	1    2950 2850
@@
 F 0 "R26" V 3780 2950 50  0000 C CNN
 F 1 "22" V 3700 2950 50  0000 C CNN
-F 2 "Resistors_SMD:R_0201" V 3630 2950 50  0001 C CNN
+F 2 "Resistors_SMD:R_0402" V 3630 2950 50  0001 C CNN
 F 3 "" H 3700 2950 50  0000 C CNN
 	1    3700 2950
@@
 F 0 "R19" V 3530 3050 50  0000 C CNN
 F 1 "22" V 3450 3050 50  0000 C CNN
-F 2 "Resistors_SMD:R_0201" V 3380 3050 50  0001 C CNN
+F 2 "Resistors_SMD:R_0402" V 3380 3050 50  0001 C CNN
 F 3 "" H 3450 3050 50  0000 C CNN
 	1    3450 3050
@@
 F 0 "R13" V 3280 3150 50  0000 C CNN
 F 1 "22" V 3200 3150 50  0000 C CNN
-F 2 "Resistors_SMD:R_0201" V 3130 3150 50  0001 C CNN
+F 2 "Resistors_SMD:R_0402" V 3130 3150 50  0001 C CNN
 F 3 "" H 3200 3150 50  0000 C CNN
 	1    3200 3150
@@
 F 0 "R7" V 3030 3250 50  0000 C CNN
 F 1 "22" V 2950 3250 50  0000 C CNN
-F 2 "Resistors_SMD:R_0201" V 2880 3250 50  0001 C CNN
+F 2 "Resistors_SMD:R_0402" V 2880 3250 50  0001 C CNN
 F 3 "" H 2950 3250 50  0000 C CNN
 	1    2950 3250
@@
 F 0 "R27" V 3780 3350 50  0000 C CNN
 F 1 "22" V 3700 3350 50  0000 C CNN
-F 2 "Resistors_SMD:R_0201" V 3630 3350 50  0001 C CNN
+F 2 "Resistors_SMD:R_0402" V 3630 3350 50  0001 C CNN
 F 3 "" H 3700 3350 50  0000 C CNN
 	1    3700 3350
@@
 F 0 "R20" V 3530 3450 50  0000 C CNN
 F 1 "22" V 3450 3450 50  0000 C CNN
-F 2 "Resistors_SMD:R_0201" V 3380 3450 50  0001 C CNN
+F 2 "Resistors_SMD:R_0402" V 3380 3450 50  0001 C CNN
 F 3 "" H 3450 3450 50  0000 C CNN
 	1    3450 3450
@@
 F 0 "R14" V 3280 3550 50  0000 C CNN
 F 1 "22" V 3200 3550 50  0000 C CNN
-F 2 "Resistors_SMD:R_0201" V 3130 3550 50  0001 C CNN
+F 2 "Resistors_SMD:R_0402" V 3130 3550 50  0001 C CNN
 F 3 "" H 3200 3550 50  0000 C CNN
 	1    3200 3550
@@
 F 0 "R8" V 3030 3650 50  0000 C CNN
 F 1 "22" V 2950 3650 50  0000 C CNN
-F 2 "Resistors_SMD:R_0201" V 2880 3650 50  0001 C CNN
+F 2 "Resistors_SMD:R_0402" V 2880 3650 50  0001 C CNN
 F 3 "" H 2950 3650 50  0000 C CNN
 	1    2950 3650
@@
 F 0 "R28" V 3780 3750 50  0000 C CNN
 F 1 "22" V 3700 3750 50  0000 C CNN
-F 2 "Resistors_SMD:R_0201" V 3630 3750 50  0001 C CNN
+F 2 "Resistors_SMD:R_0402" V 3630 3750 50  0001 C CNN
 F 3 "" H 3700 3750 50  0000 C CNN
 	1    3700 3750
@@
 F 0 "R21" V 3530 3850 50  0000 C CNN
 F 1 "22" V 3450 3850 50  0000 C CNN
-F 2 "Resistors_SMD:R_0201" V 3380 3850 50  0001 C CNN
+F 2 "Resistors_SMD:R_0402" V 3380 3850 50  0001 C CNN
 F 3 "" H 3450 3850 50  0000 C CNN
 	1    3450 3850
@@
 F 0 "R15" V 3280 3950 50  0000 C CNN
 F 1 "22" V 3200 3950 50  0000 C CNN
-F 2 "Resistors_SMD:R_0201" V 3130 3950 50  0001 C CNN
+F 2 "Resistors_SMD:R_0402" V 3130 3950 50  0001 C CNN
 F 3 "" H 3200 3950 50  0000 C CNN
 	1    3200 3950
@@
 F 0 "R9" V 3030 4050 50  0000 C CNN
 F 1 "22" V 2950 4050 50  0000 C CNN
-F 2 "Resistors_SMD:R_0201" V 2880 4050 50  0001 C CNN
+F 2 "Resistors_SMD:R_0402" V 2880 4050 50  0001 C CNN
 F 3 "" H 2950 4050 50  0000 C CNN
 	1    2950 4050
@@
 F 0 "R29" V 3780 4150 50  0000 C CNN
 F 1 "22" V 3700 4150 50  0000 C CNN
-F 2 "Resistors_SMD:R_0201" V 3630 4150 50  0001 C CNN
+F 2 "Resistors_SMD:R_0402" V 3630 4150 50  0001 C CNN
 F 3 "" H 3700 4150 50  0000 C CNN
 	1    3700 4150
@@
 F 0 "R22" V 3530 4250 50  0000 C CNN
 F 1 "22" V 3450 4250 50  0000 C CNN
-F 2 "Resistors_SMD:R_0201" V 3380 4250 50  0001 C CNN
+F 2 "Resistors_SMD:R_0402" V 3380 4250 50  0001 C CNN
 F 3 "" H 3450 4250 50  0000 C CNN
 	1    3450 4250
