File: gpif2.sch (KiCad schematic (older format))
At the start: 38 parts, among them Q3 IRLML2502, SW1 TL6215RF200BDT, U1 xc7a50tftg256

Commit message: screen attached!
Connections:
- net GND: no longer U1.P9 (IO_L18N_T2_A11_D27_14), U1.R10 (IO_L17P_T2_A14_D30_14), U1.T10 (IO_L22N_T3_A04_D20_14)
- net TEMPO_LED: no longer U1.T5 (IO_L23N_T3_A02_D18_14)
- net I2S_ADCSD: no longer names the net of U1.T13 (IO_L16N_T2_A15_D31_14)
- net I2S_BCLK: no longer names the net of U1.N11 (IO_L13P_T2_MRCC_14)
- net I2S_LRCLK: no longer names the net of U1.P14 (IO_L12N_T1_MRCC_14)
- new net LED_1B_CTRL: U1.P9 (IO_L18N_T2_A11_D27_14)
- new net LED_1G_CTRL: U1.T10 (IO_L22N_T3_A04_D20_14)
- new net LED_1R_CTRL: U1.R10 (IO_L17P_T2_A14_D30_14)
- no-connect marks 3 -> 7
Changed lines of the file:
@@
 $Descr A4 11693 8268
 encoding utf-8
-Sheet 4 15
+Sheet 4 14
 Title ""
 Date ""
@@
 $EndComp
 $Comp
-L +1.8V #PWR013
+L +1.8V #PWR010
 U 1 1 585C5E93
 P 5400 6400
-F 0 "#PWR013" H 5400 6540 20  0001 C CNN
+F 0 "#PWR010" H 5400 6540 20  0001 C CNN
 F 1 "+1.8V" H 5400 6510 30  0000 C CNN
 F 2 "" H 5400 6400 60  0001 C CNN
@@
 Connection ~ 5150 7200
 $Comp
-L GND #PWR014
+L GND #PWR011
 U 1 1 586C88E4
 P 5400 7300
-F 0 "#PWR014" H 5400 7050 50  0001 C CNN
+F 0 "#PWR011" H 5400 7050 50  0001 C CNN
 F 1 "GND" H 5400 7150 50  0000 C CNN
 F 2 "" H 5400 7300 50  0000 C CNN
@@
 	1    0    0    -1
 $EndComp
-Text GLabel 5950 3950 0    60   Input ~ 0
-I2S_LRCLK
-Text GLabel 5950 4250 0    60   Input ~ 0
-I2S_BCLK
 Text GLabel 5950 4550 0    60   Output ~ 0
 I2S_DACSD
@@
 $EndComp
 $Comp
-L GND #PWR015
+L GND #PWR012
 U 1 1 587AD7CC
 P 8650 3550
-F 0 "#PWR015" H 8650 3300 50  0001 C CNN
+F 0 "#PWR012" H 8650 3300 50  0001 C CNN
 F 1 "GND" H 8650 3400 50  0000 C CNN
 F 2 "" H 8650 3550 50  0000 C CNN
@@
 $EndComp
 $Comp
-L GND #PWR016
+L GND #PWR013
 U 1 1 587B04F2
 P 8850 4400
-F 0 "#PWR016" H 8850 4150 50  0001 C CNN
+F 0 "#PWR013" H 8850 4150 50  0001 C CNN
 F 1 "GND" H 8850 4250 50  0000 C CNN
 F 2 "" H 8850 4400 50  0000 C CNN
@@
 	9700 3650 9900 3650
 $Comp
-L +5V #PWR017
+L +5V #PWR014
 U 1 1 587B1756
 P 10400 3650
-F 0 "#PWR017" H 10400 3500 50  0001 C CNN
+F 0 "#PWR014" H 10400 3500 50  0001 C CNN
 F 1 "+5V" H 10400 3790 50  0000 C CNN
 F 2 "" H 10400 3650 50  0000 C CNN
@@
 Text GLabel 10050 3400 2    60   Output ~ 0
 TEMPO_SW
-Text GLabel 5950 6150 0    60   Output ~ 0
-TEMPO_LED
 Text GLabel 9150 4150 2    60   Input ~ 0
 TEMPO_LED
-Text GLabel 5950 4750 0    60   Input ~ 0
-I2S_ADCSD
 $Comp
 L R R30
@@
 	9700 3400 10050 3400
 $Comp
-L +1.8V #PWR018
+L +1.8V #PWR015
 U 1 1 588410AE
 P 9850 2900
-F 0 "#PWR018" H 9850 3040 20  0001 C CNN
+F 0 "#PWR015" H 9850 3040 20  0001 C CNN
 F 1 "+1.8V" H 9850 3010 30  0000 C CNN
 F 2 "" H 9850 2900 60  0001 C CNN
@@
 GD_1T
 $Comp
-L GND #PWR019
+L GND #PWR016
 U 1 1 58945BF9
 P 5950 4150
-F 0 "#PWR019" H 5950 3900 50  0001 C CNN
+F 0 "#PWR016" H 5950 3900 50  0001 C CNN
 F 1 "GND" H 5950 4000 50  0000 C CNN
 F 2 "" H 5950 4150 50  0000 C CNN
@@
 $EndComp
 $Comp
-L GND #PWR020
+L GND #PWR017
 U 1 1 589461C0
 P 5950 4450
-F 0 "#PWR020" H 5950 4200 50  0001 C CNN
+F 0 "#PWR017" H 5950 4200 50  0001 C CNN
 F 1 "GND" H 5950 4300 50  0000 C CNN
 F 2 "" H 5950 4450 50  0000 C CNN
@@
 $EndComp
 $Comp
-L GND #PWR021
-U 1 1 58946355
-P 5950 5050
-F 0 "#PWR021" H 5950 4800 50  0001 C CNN
-F 1 "GND" H 5950 4900 50  0000 C CNN
-F 2 "" H 5950 5050 50  0000 C CNN
-F 3 "" H 5950 5050 50  0000 C CNN
-	1    5950 5050
-	0    1    1    0
-$EndComp
-$Comp
-L GND #PWR022
-U 1 1 58946634
-P 5950 5950
-F 0 "#PWR022" H 5950 5700 50  0001 C CNN
-F 1 "GND" H 5950 5800 50  0000 C CNN
-F 2 "" H 5950 5950 50  0000 C CNN
-F 3 "" H 5950 5950 50  0000 C CNN
-	1    5950 5950
-	0    1    1    0
-$EndComp
-$Comp
-L GND #PWR023
+L GND #PWR018
 U 1 1 589483E2
 P 5950 1650
-F 0 "#PWR023" H 5950 1400 50  0001 C CNN
+F 0 "#PWR018" H 5950 1400 50  0001 C CNN
 F 1 "GND" H 5950 1500 50  0000 C CNN
 F 2 "" H 5950 1650 50  0000 C CNN
@@
 $EndComp
 $Comp
-L GND #PWR024
+L GND #PWR019
 U 1 1 58948C63
 P 5950 6450
-F 0 "#PWR024" H 5950 6200 50  0001 C CNN
+F 0 "#PWR019" H 5950 6200 50  0001 C CNN
 F 1 "GND" H 5950 6300 50  0000 C CNN
 F 2 "" H 5950 6450 50  0000 C CNN
@@
 $EndComp
 $Comp
-L GND #PWR025
+L GND #PWR020
 U 1 1 5894C026
 P 5950 6350
-F 0 "#PWR025" H 5950 6100 50  0001 C CNN
+F 0 "#PWR020" H 5950 6100 50  0001 C CNN
 F 1 "GND" H 5950 6200 50  0000 C CNN
 F 2 "" H 5950 6350 50  0000 C CNN
@@
 $EndComp
 $Comp
-L GND #PWR026
+L GND #PWR021
 U 1 1 5894C0A3
 P 5950 5650
-F 0 "#PWR026" H 5950 5400 50  0001 C CNN
+F 0 "#PWR021" H 5950 5400 50  0001 C CNN
 F 1 "GND" H 5950 5500 50  0000 C CNN
 F 2 "" H 5950 5650 50  0000 C CNN
@@
 $EndComp
 $Comp
-L GND #PWR027
+L GND #PWR022
 U 1 1 5894C120
 P 5950 5550
-F 0 "#PWR027" H 5950 5300 50  0001 C CNN
+F 0 "#PWR022" H 5950 5300 50  0001 C CNN
 F 1 "GND" H 5950 5400 50  0000 C CNN
 F 2 "" H 5950 5550 50  0000 C CNN
@@
 $EndComp
 $Comp
-L GND #PWR028
+L GND #PWR023
 U 1 1 5894C19D
 P 5950 5250
-F 0 "#PWR028" H 5950 5000 50  0001 C CNN
+F 0 "#PWR023" H 5950 5000 50  0001 C CNN
 F 1 "GND" H 5950 5100 50  0000 C CNN
 F 2 "" H 5950 5250 50  0000 C CNN
@@
 $EndComp
 $Comp
-L GND #PWR029
-U 1 1 5894C21A
-P 5950 5150
-F 0 "#PWR029" H 5950 4900 50  0001 C CNN
-F 1 "GND" H 5950 5000 50  0000 C CNN
-F 2 "" H 5950 5150 50  0000 C CNN
-F 3 "" H 5950 5150 50  0000 C CNN
-	1    5950 5150
-	0    1    1    0
-$EndComp
-$Comp
-L GND #PWR030
+L GND #PWR024
 U 1 1 5894C331
 P 5950 6050
-F 0 "#PWR030" H 5950 5800 50  0001 C CNN
+F 0 "#PWR024" H 5950 5800 50  0001 C CNN
 F 1 "GND" H 5950 5900 50  0000 C CNN
 F 2 "" H 5950 6050 50  0000 C CNN
@@
 $EndComp
 $Comp
-L GND #PWR031
+L GND #PWR025
 U 1 1 5894CCAA
 P 5950 5350
-F 0 "#PWR031" H 5950 5100 50  0001 C CNN
+F 0 "#PWR025" H 5950 5100 50  0001 C CNN
 F 1 "GND" H 5950 5200 50  0000 C CNN
 F 2 "" H 5950 5350 50  0000 C CNN
@@
 $EndComp
 $Comp
-L GND #PWR032
+L GND #PWR026
 U 1 1 5894CD27
 P 5950 5450
-F 0 "#PWR032" H 5950 5200 50  0001 C CNN
+F 0 "#PWR026" H 5950 5200 50  0001 C CNN
 F 1 "GND" H 5950 5300 50  0000 C CNN
 F 2 "" H 5950 5450 50  0000 C CNN
@@
 Text GLabel 5950 1750 0    60   Input ~ 0
 SPI_MISO
+Text GLabel 5950 5150 0    60   Output ~ 0
+LED_1B_CTRL
+Text GLabel 5950 5950 0    60   Output ~ 0
+LED_1G_CTRL
+NoConn ~ 5950 6150
+Text GLabel 5950 5050 0    60   Output ~ 0
+LED_1R_CTRL
+NoConn ~ 5950 4750
+NoConn ~ 5950 4250
+NoConn ~ 5950 3950
 $EndSCHEMATC

Commit message: using BOMs AWAY to create BOM
Parts:
- C2: MFR (none) -> Murata Manufacturing Co Ltd; MPN (none) -> GRM32ER70J476ME20L
- C3, C4: MFR (none) -> Murata; MPN (none) -> GRM21BR61A475KA73L
- C5, C6, C7, C8: MFR (none) -> Murata; MPN (none) -> GRM188R71C474KA88D
- Q3: MFR (none) -> Infineon Technologies AG; MPN (none) -> IRLML2502TRPBF
- R10, R11, R12, R13, R14, R15, R16, R17, R18, R19, R20, R21, R22, R23, R24, R25, R26, R27, R28, R29, R30, R31, R6, R7, R8, R9: MFR (none) -> Vishay Dale; MPN (none) -> CRCW040222R0FKED
- R32: MFR (none) -> Vishay Dale; MPN (none) -> CRCW040210K0FKED
- R33: MFR (none) -> Vishay Dale; MPN (none) -> CRCW0402150RFKED
- SW1: MFR (none) -> E-Switch Inc; MPN (none) -> TL6215RF200BDT
- U1: MFR (none) -> Xilinx; MPN (none) -> XC7A50T-1FTG256C

Commit message: just added NOTE field to BOMS AWAY
Parts:
- C2: SPN (none) -> 490-6542-1-ND; SPR (none) -> Digikey
- C3, C4: SPN (none) -> 490-9750-1-ND; SPR (none) -> Digikey
- C5, C6, C7, C8: SPN (none) -> 490-3295-1-ND; SPR (none) -> Digikey
Changed lines of the file:
@@
 F 4 "Murata Manufacturing Co Ltd" H 0 0 50 0001 C CNN "MFR"
 F 5 "GRM32ER70J476ME20L" H 0 0 50 0001 C CNN "MPN"
-F 6 "" H 0 0 50 0001 C CNN "SPR"
-F 7 "" H 0 0 50 0001 C CNN "SPN"
+F 6 "Digikey" H 0 0 50 0001 C CNN "SPR"
+F 7 "490-6542-1-ND" H 0 0 50 0001 C CNN "SPN"
 F 8 "" H 0 0 50 0001 C CNN "SPURL"
 	1    4900 7000
@@
 F 4 "Murata" H 0 0 50 0001 C CNN "MFR"
 F 5 "GRM21BR61A475KA73L" H 0 0 50 0001 C CNN "MPN"
-F 6 "" H 0 0 50 0001 C CNN "SPR"
-F 7 "" H 0 0 50 0001 C CNN "SPN"
+F 6 "Digikey" H 0 0 50 0001 C CNN "SPR"
+F 7 "490-9750-1-ND" H 0 0 50 0001 C CNN "SPN"
 F 8 "" H 0 0 50 0001 C CNN "SPURL"
 	1    5150 7000
@@
 F 4 "Murata" H 0 0 50 0001 C CNN "MFR"
 F 5 "GRM21BR61A475KA73L" H 0 0 50 0001 C CNN "MPN"
-F 6 "" H 0 0 50 0001 C CNN "SPR"
-F 7 "" H 0 0 50 0001 C CNN "SPN"
+F 6 "Digikey" H 0 0 50 0001 C CNN "SPR"
+F 7 "490-9750-1-ND" H 0 0 50 0001 C CNN "SPN"
 F 8 "" H 0 0 50 0001 C CNN "SPURL"
 	1    5400 7000
@@
 F 4 "Murata" H 0 0 50 0001 C CNN "MFR"
 F 5 "GRM188R71C474KA88D" H 0 0 50 0001 C CNN "MPN"
-F 6 "" H 0 0 50 0001 C CNN "SPR"
-F 7 "" H 0 0 50 0001 C CNN "SPN"
+F 6 "Digikey" H 0 0 50 0001 C CNN "SPR"
+F 7 "490-3295-1-ND" H 0 0 50 0001 C CNN "SPN"
 F 8 "" H 0 0 50 0001 C CNN "SPURL"
 	1    5650 7000
@@
 F 4 "Murata" H 0 0 50 0001 C CNN "MFR"
 F 5 "GRM188R71C474KA88D" H 0 0 50 0001 C CNN "MPN"
-F 6 "" H 0 0 50 0001 C CNN "SPR"
-F 7 "" H 0 0 50 0001 C CNN "SPN"
+F 6 "Digikey" H 0 0 50 0001 C CNN "SPR"
+F 7 "490-3295-1-ND" H 0 0 50 0001 C CNN "SPN"
 F 8 "" H 0 0 50 0001 C CNN "SPURL"
 	1    5900 7000
@@
 F 4 "Murata" H 0 0 50 0001 C CNN "MFR"
 F 5 "GRM188R71C474KA88D" H 0 0 50 0001 C CNN "MPN"
-F 6 "" H 0 0 50 0001 C CNN "SPR"
-F 7 "" H 0 0 50 0001 C CNN "SPN"
+F 6 "Digikey" H 0 0 50 0001 C CNN "SPR"
+F 7 "490-3295-1-ND" H 0 0 50 0001 C CNN "SPN"
 F 8 "" H 0 0 50 0001 C CNN "SPURL"
 	1    6150 7000
@@
 F 4 "Murata" H 0 0 50 0001 C CNN "MFR"
 F 5 "GRM188R71C474KA88D" H 0 0 50 0001 C CNN "MPN"
-F 6 "" H 0 0 50 0001 C CNN "SPR"
-F 7 "" H 0 0 50 0001 C CNN "SPN"
+F 6 "Digikey" H 0 0 50 0001 C CNN "SPR"
+F 7 "490-3295-1-ND" H 0 0 50 0001 C CNN "SPN"
 F 8 "" H 0 0 50 0001 C CNN "SPURL"
 	1    6400 7000

Commit message: Complete BOM. all resistors now 0402
Parts:
- Q3: SPN (none) -> IRLML2502PBFCT-ND; SPR (none) -> Digikey
- R10, R11, R12, R13, R14, R15, R16, R17, R18, R19, R20, R21, R22, R23, R24, R25, R26, R27, R28, R29, R30, R31, R6, R7, R8, R9: MFR Vishay Dale -> Yageo; MPN CRCW040222R0FKED -> RC0402FR-0722RL; SPN (none) -> 311-22.0LRTR-ND; SPR (none) -> Digikey
- R32: MFR Vishay Dale -> Yageo; MPN CRCW040210K0FKED -> RC0402FR-0710KL; SPN (none) -> 311-10.0KLRTR-ND; SPR (none) -> Digikey
- R33: MFR Vishay Dale -> Yageo; MPN CRCW0402150RFKED -> RC0402FR-07150RL; SPN (none) -> 311-150LRTR-ND; SPR (none) -> Digikey
- SW1: SPN (none) -> EG5162-ND; SPR (none) -> Digikey
- U1: SPN (none) -> 122-1916-ND; SPR (none) -> Digikey
