File: FPGA_POWER.sch (KiCad schematic (older format))
At the start: 18 parts, among them U1 xc7a50tftg256

Commit message: using BOMs AWAY to create BOM
Parts:
- C10, C11, C12, C13, C14, C16, C18, C23, C9: MFR (none) -> Murata; MPN (none) -> GRM188R71C474KA88D
- C15, C17, C20, C21, C22: MFR (none) -> Murata; MPN (none) -> GRM21BR61A475KA73L
- C19: MFR (none) -> Murata Manufacturing Co Ltd; MPN (none) -> GRM32ER70J476ME20L
- C24: MFR (none) -> AVX Corporation; MPN (none) -> F950G337MAAAQ2
- C25: MFR (none) -> TAIYO YUDEN; MPN (none) -> JMK325ABJ107MM-P
- U1: MFR (none) -> Xilinx; MPN (none) -> XC7A50T-1FTG256C

Commit message: just added NOTE field to BOMS AWAY
Parts:
- C10, C11, C12, C13, C14, C16, C18, C23, C9: SPN (none) -> 490-3295-1-ND; SPR (none) -> Digikey
- C15, C17, C20, C21, C22: SPN (none) -> 490-9750-1-ND; SPR (none) -> Digikey
- C19: SPN (none) -> 490-6542-1-ND; SPR (none) -> Digikey
- C24: SPN (none) -> 478-8378-1-ND; SPR (none) -> Digikey
- C25: SPN (none) -> 587-4313-1-ND; SPR (none) -> Digikey
Changed lines of the file:
@@
 F 4 "Murata" H 0 0 50 0001 C CNN "MFR"
 F 5 "GRM21BR61A475KA73L" H 0 0 50 0001 C CNN "MPN"
-F 6 "" H 0 0 50 0001 C CNN "SPR"
-F 7 "" H 0 0 50 0001 C CNN "SPN"
+F 6 "Digikey" H 0 0 50 0001 C CNN "SPR"
+F 7 "490-9750-1-ND" H 0 0 50 0001 C CNN "SPN"
 F 8 "" H 0 0 50 0001 C CNN "SPURL"
 	1    3050 5750
@@
 F 4 "Murata" H 0 0 50 0001 C CNN "MFR"
 F 5 "GRM21BR61A475KA73L" H 0 0 50 0001 C CNN "MPN"
-F 6 "" H 0 0 50 0001 C CNN "SPR"
-F 7 "" H 0 0 50 0001 C CNN "SPN"
+F 6 "Digikey" H 0 0 50 0001 C CNN "SPR"
+F 7 "490-9750-1-ND" H 0 0 50 0001 C CNN "SPN"
 F 8 "" H 0 0 50 0001 C CNN "SPURL"
 	1    2800 5750
@@
 F 4 "Murata" H 0 0 50 0001 C CNN "MFR"
 F 5 "GRM21BR61A475KA73L" H 0 0 50 0001 C CNN "MPN"
-F 6 "" H 0 0 50 0001 C CNN "SPR"
-F 7 "" H 0 0 50 0001 C CNN "SPN"
+F 6 "Digikey" H 0 0 50 0001 C CNN "SPR"
+F 7 "490-9750-1-ND" H 0 0 50 0001 C CNN "SPN"
 F 8 "" H 0 0 50 0001 C CNN "SPURL"
 	1    2550 5750
@@
 F 4 "Murata" H 0 0 50 0001 C CNN "MFR"
 F 5 "GRM188R71C474KA88D" H 0 0 50 0001 C CNN "MPN"
-F 6 "" H 0 0 50 0001 C CNN "SPR"
-F 7 "" H 0 0 50 0001 C CNN "SPN"
+F 6 "Digikey" H 0 0 50 0001 C CNN "SPR"
+F 7 "490-3295-1-ND" H 0 0 50 0001 C CNN "SPN"
 F 8 "" H 0 0 50 0001 C CNN "SPURL"
 	1    2200 5750
@@
 F 4 "Murata" H 0 0 50 0001 C CNN "MFR"
 F 5 "GRM188R71C474KA88D" H 0 0 50 0001 C CNN "MPN"
-F 6 "" H 0 0 50 0001 C CNN "SPR"
-F 7 "" H 0 0 50 0001 C CNN "SPN"
+F 6 "Digikey" H 0 0 50 0001 C CNN "SPR"
+F 7 "490-3295-1-ND" H 0 0 50 0001 C CNN "SPN"
 F 8 "" H 0 0 50 0001 C CNN "SPURL"
 	1    1950 5750
@@
 F 4 "Murata" H 0 0 50 0001 C CNN "MFR"
 F 5 "GRM188R71C474KA88D" H 0 0 50 0001 C CNN "MPN"
-F 6 "" H 0 0 50 0001 C CNN "SPR"
-F 7 "" H 0 0 50 0001 C CNN "SPN"
+F 6 "Digikey" H 0 0 50 0001 C CNN "SPR"
+F 7 "490-3295-1-ND" H 0 0 50 0001 C CNN "SPN"
 F 8 "" H 0 0 50 0001 C CNN "SPURL"
 	1    1700 5750
@@
 F 4 "Murata" H 0 0 50 0001 C CNN "MFR"
 F 5 "GRM188R71C474KA88D" H 0 0 50 0001 C CNN "MPN"
-F 6 "" H 0 0 50 0001 C CNN "SPR"
-F 7 "" H 0 0 50 0001 C CNN "SPN"
+F 6 "Digikey" H 0 0 50 0001 C CNN "SPR"
+F 7 "490-3295-1-ND" H 0 0 50 0001 C CNN "SPN"
 F 8 "" H 0 0 50 0001 C CNN "SPURL"
 	1    1200 5750
@@
 F 4 "Murata" H 0 0 50 0001 C CNN "MFR"
 F 5 "GRM188R71C474KA88D" H 0 0 50 0001 C CNN "MPN"
-F 6 "" H 0 0 50 0001 C CNN "SPR"
-F 7 "" H 0 0 50 0001 C CNN "SPN"
+F 6 "Digikey" H 0 0 50 0001 C CNN "SPR"
+F 7 "490-3295-1-ND" H 0 0 50 0001 C CNN "SPN"
 F 8 "" H 0 0 50 0001 C CNN "SPURL"
 	1    1450 5750
@@
 F 4 "TAIYO YUDEN" H 0 0 50 0001 C CNN "MFR"
 F 5 "JMK325ABJ107MM-P" H 0 0 50 0001 C CNN "MPN"
-F 6 "" H 0 0 50 0001 C CNN "SPR"
-F 7 "" H 0 0 50 0001 C CNN "SPN"
+F 6 "Digikey" H 0 0 50 0001 C CNN "SPR"
+F 7 "587-4313-1-ND" H 0 0 50 0001 C CNN "SPN"
 F 8 "" H 0 0 50 0001 C CNN "SPURL"
 	1    3500 5050
@@
 F 4 "Murata" H 0 0 50 0001 C CNN "MFR"
 F 5 "GRM188R71C474KA88D" H 0 0 50 0001 C CNN "MPN"
-F 6 "" H 0 0 50 0001 C CNN "SPR"
-F 7 "" H 0 0 50 0001 C CNN "SPN"
+F 6 "Digikey" H 0 0 50 0001 C CNN "SPR"
+F 7 "490-3295-1-ND" H 0 0 50 0001 C CNN "SPN"
 F 8 "" H 0 0 50 0001 C CNN "SPURL"
 	1    3150 5050
@@
 F 4 "Murata Manufacturing Co Ltd" H 0 0 50 0001 C CNN "MFR"
 F 5 "GRM32ER70J476ME20L" H 0 0 50 0001 C CNN "MPN"
-F 6 "" H 0 0 50 0001 C CNN "SPR"
-F 7 "" H 0 0 50 0001 C CNN "SPN"
+F 6 "Digikey" H 0 0 50 0001 C CNN "SPR"
+F 7 "490-6542-1-ND" H 0 0 50 0001 C CNN "SPN"
 F 8 "" H 0 0 50 0001 C CNN "SPURL"
 	1    2450 4700
@@
 F 4 "Murata" H 0 0 50 0001 C CNN "MFR"
 F 5 "GRM21BR61A475KA73L" H 0 0 50 0001 C CNN "MPN"
-F 6 "" H 0 0 50 0001 C CNN "SPR"
-F 7 "" H 0 0 50 0001 C CNN "SPN"
+F 6 "Digikey" H 0 0 50 0001 C CNN "SPR"
+F 7 "490-9750-1-ND" H 0 0 50 0001 C CNN "SPN"
 F 8 "" H 0 0 50 0001 C CNN "SPURL"
 	1    2150 4700
@@
 F 4 "Murata" H 0 0 50 0001 C CNN "MFR"
 F 5 "GRM21BR61A475KA73L" H 0 0 50 0001 C CNN "MPN"
-F 6 "" H 0 0 50 0001 C CNN "SPR"
-F 7 "" H 0 0 50 0001 C CNN "SPN"
+F 6 "Digikey" H 0 0 50 0001 C CNN "SPR"
+F 7 "490-9750-1-ND" H 0 0 50 0001 C CNN "SPN"
 F 8 "" H 0 0 50 0001 C CNN "SPURL"
 	1    1900 4700
@@
 F 4 "Murata" H 0 0 50 0001 C CNN "MFR"
 F 5 "GRM188R71C474KA88D" H 0 0 50 0001 C CNN "MPN"
-F 6 "" H 0 0 50 0001 C CNN "SPR"
-F 7 "" H 0 0 50 0001 C CNN "SPN"
+F 6 "Digikey" H 0 0 50 0001 C CNN "SPR"
+F 7 "490-3295-1-ND" H 0 0 50 0001 C CNN "SPN"
 F 8 "" H 0 0 50 0001 C CNN "SPURL"
 	1    1650 4700
@@
 F 4 "Murata" H 0 0 50 0001 C CNN "MFR"
 F 5 "GRM188R71C474KA88D" H 0 0 50 0001 C CNN "MPN"
-F 6 "" H 0 0 50 0001 C CNN "SPR"
-F 7 "" H 0 0 50 0001 C CNN "SPN"
+F 6 "Digikey" H 0 0 50 0001 C CNN "SPR"
+F 7 "490-3295-1-ND" H 0 0 50 0001 C CNN "SPN"
 F 8 "" H 0 0 50 0001 C CNN "SPURL"
 	1    1400 4700
@@
 F 4 "Murata" H 0 0 50 0001 C CNN "MFR"
 F 5 "GRM188R71C474KA88D" H 0 0 50 0001 C CNN "MPN"
-F 6 "" H 0 0 50 0001 C CNN "SPR"
-F 7 "" H 0 0 50 0001 C CNN "SPN"
+F 6 "Digikey" H 0 0 50 0001 C CNN "SPR"
+F 7 "490-3295-1-ND" H 0 0 50 0001 C CNN "SPN"
 F 8 "" H 0 0 50 0001 C CNN "SPURL"
 	1    1150 4700
@@
 F 4 "AVX Corporation" H 0 0 50 0001 C CNN "MFR"
 F 5 "F950G337MAAAQ2" H 0 0 50 0001 C CNN "MPN"
-F 6 "" H 0 0 50 0001 C CNN "SPR"
-F 7 "" H 0 0 50 0001 C CNN "SPN"
+F 6 "Digikey" H 0 0 50 0001 C CNN "SPR"
+F 7 "478-8378-1-ND" H 0 0 50 0001 C CNN "SPN"
 F 8 "" H 0 0 50 0001 C CNN "SPURL"
 	1    3350 5750

Commit message: Complete BOM. all resistors now 0402
Parts:
- U1: SPN (none) -> 122-1916-ND; SPR (none) -> Digikey
