File: power.sch (KiCad schematic (older format))
At the start: 17 parts, among them U4 SC189 - 3.3V, U5 SC189 - 1.0V, U6 SC189 - 1.2V, U7 SC189 - 1.8V

Commit message: using BOMs AWAY to create BOM
Parts:
- C89, C90, C91, C92, C93, C94, C95, C96: MFR (none) -> Murata; MPN (none) -> GRM21BR61A106KE19L
- L1, L2, L3, L4: MFR (none) -> Murata; MPN (none) -> LQH43PN2R2M26L
- U4: MFR (none) -> Semtech Corporation; MPN (none) -> SC189ZSKTRT
- U5: MFR (none) -> Semtech Corporation; MPN (none) -> SC189ASKTRT
- U6: MFR (none) -> Semtech Corporation; MPN (none) -> SC189CSKTRT
- U7: MFR (none) -> Semtech Corporation; MPN (none) -> SC189LSKTRT

Commit message: just added NOTE field to BOMS AWAY
Parts:
- C89, C90, C91, C92, C93, C94, C95, C96: SPN (none) -> 490-1709-1-ND; SPR (none) -> Digikey
- L1, L2, L3, L4: SPN (none) -> 490-12049-1-ND; SPR (none) -> Digikey
Changed lines of the file:
@@
 F 4 "Murata" H 0 0 50 0001 C CNN "MFR"
 F 5 "GRM21BR61A106KE19L" H 0 0 50 0001 C CNN "MPN"
-F 6 "" H 0 0 50 0001 C CNN "SPR"
-F 7 "" H 0 0 50 0001 C CNN "SPN"
+F 6 "Digikey" H 0 0 50 0001 C CNN "SPR"
+F 7 "490-1709-1-ND" H 0 0 50 0001 C CNN "SPN"
 F 8 "" H 0 0 50 0001 C CNN "SPURL"
 	1    3600 2950
@@
 F 4 "Murata" H 0 0 50 0001 C CNN "MFR"
 F 5 "GRM21BR61A106KE19L" H 0 0 50 0001 C CNN "MPN"
-F 6 "" H 0 0 50 0001 C CNN "SPR"
-F 7 "" H 0 0 50 0001 C CNN "SPN"
+F 6 "Digikey" H 0 0 50 0001 C CNN "SPR"
+F 7 "490-1709-1-ND" H 0 0 50 0001 C CNN "SPN"
 F 8 "" H 0 0 50 0001 C CNN "SPURL"
 	1    7250 2950
@@
 F 4 "Murata" H 0 0 50 0001 C CNN "MFR"
 F 5 "GRM21BR61A106KE19L" H 0 0 50 0001 C CNN "MPN"
-F 6 "" H 0 0 50 0001 C CNN "SPR"
-F 7 "" H 0 0 50 0001 C CNN "SPN"
+F 6 "Digikey" H 0 0 50 0001 C CNN "SPR"
+F 7 "490-1709-1-ND" H 0 0 50 0001 C CNN "SPN"
 F 8 "" H 0 0 50 0001 C CNN "SPURL"
 	1    7250 4800
@@
 F 4 "Murata" H 0 0 50 0001 C CNN "MFR"
 F 5 "GRM21BR61A106KE19L" H 0 0 50 0001 C CNN "MPN"
-F 6 "" H 0 0 50 0001 C CNN "SPR"
-F 7 "" H 0 0 50 0001 C CNN "SPN"
+F 6 "Digikey" H 0 0 50 0001 C CNN "SPR"
+F 7 "490-1709-1-ND" H 0 0 50 0001 C CNN "SPN"
 F 8 "" H 0 0 50 0001 C CNN "SPURL"
 	1    3600 4800
@@
 F 4 "Murata" H 0 0 50 0001 C CNN "MFR"
 F 5 "GRM21BR61A106KE19L" H 0 0 50 0001 C CNN "MPN"
-F 6 "" H 0 0 50 0001 C CNN "SPR"
-F 7 "" H 0 0 50 0001 C CNN "SPN"
+F 6 "Digikey" H 0 0 50 0001 C CNN "SPR"
+F 7 "490-1709-1-ND" H 0 0 50 0001 C CNN "SPN"
 F 8 "" H 0 0 50 0001 C CNN "SPURL"
 	1    6200 3250
@@
 F 4 "Murata" H 0 0 50 0001 C CNN "MFR"
 F 5 "GRM21BR61A106KE19L" H 0 0 50 0001 C CNN "MPN"
-F 6 "" H 0 0 50 0001 C CNN "SPR"
-F 7 "" H 0 0 50 0001 C CNN "SPN"
+F 6 "Digikey" H 0 0 50 0001 C CNN "SPR"
+F 7 "490-1709-1-ND" H 0 0 50 0001 C CNN "SPN"
 F 8 "" H 0 0 50 0001 C CNN "SPURL"
 	1    6200 5100
@@
 F 4 "Murata" H 0 0 50 0001 C CNN "MFR"
 F 5 "GRM21BR61A106KE19L" H 0 0 50 0001 C CNN "MPN"
-F 6 "" H 0 0 50 0001 C CNN "SPR"
-F 7 "" H 0 0 50 0001 C CNN "SPN"
+F 6 "Digikey" H 0 0 50 0001 C CNN "SPR"
+F 7 "490-1709-1-ND" H 0 0 50 0001 C CNN "SPN"
 F 8 "" H 0 0 50 0001 C CNN "SPURL"
 	1    10000 3250
@@
 F 4 "Murata" H 0 0 50 0001 C CNN "MFR"
 F 5 "GRM21BR61A106KE19L" H 0 0 50 0001 C CNN "MPN"
-F 6 "" H 0 0 50 0001 C CNN "SPR"
-F 7 "" H 0 0 50 0001 C CNN "SPN"
+F 6 "Digikey" H 0 0 50 0001 C CNN "SPR"
+F 7 "490-1709-1-ND" H 0 0 50 0001 C CNN "SPN"
 F 8 "" H 0 0 50 0001 C CNN "SPURL"
 	1    10000 5150
@@
 F 4 "Murata" H 0 0 50 0001 C CNN "MFR"
 F 5 "LQH43PN2R2M26L" H 0 0 50 0001 C CNN "MPN"
-F 6 "" H 0 0 50 0001 C CNN "SPR"
-F 7 "" H 0 0 50 0001 C CNN "SPN"
+F 6 "Digikey" H 0 0 50 0001 C CNN "SPR"
+F 7 "490-12049-1-ND" H 0 0 50 0001 C CNN "SPN"
 F 8 "" H 0 0 50 0001 C CNN "SPURL"
 	1    5950 3150
@@
 F 4 "Murata" H 0 0 50 0001 C CNN "MFR"
 F 5 "LQH43PN2R2M26L" H 0 0 50 0001 C CNN "MPN"
-F 6 "" H 0 0 50 0001 C CNN "SPR"
-F 7 "" H 0 0 50 0001 C CNN "SPN"
+F 6 "Digikey" H 0 0 50 0001 C CNN "SPR"
+F 7 "490-12049-1-ND" H 0 0 50 0001 C CNN "SPN"
 F 8 "" H 0 0 50 0001 C CNN "SPURL"
 	1    5950 5000
@@
 F 4 "Murata" H 0 0 50 0001 C CNN "MFR"
 F 5 "LQH43PN2R2M26L" H 0 0 50 0001 C CNN "MPN"
-F 6 "" H 0 0 50 0001 C CNN "SPR"
-F 7 "" H 0 0 50 0001 C CNN "SPN"
+F 6 "Digikey" H 0 0 50 0001 C CNN "SPR"
+F 7 "490-12049-1-ND" H 0 0 50 0001 C CNN "SPN"
 F 8 "" H 0 0 50 0001 C CNN "SPURL"
 	1    9750 5000
@@
 F 4 "Murata" H 0 0 50 0001 C CNN "MFR"
 F 5 "LQH43PN2R2M26L" H 0 0 50 0001 C CNN "MPN"
-F 6 "" H 0 0 50 0001 C CNN "SPR"
-F 7 "" H 0 0 50 0001 C CNN "SPN"
+F 6 "Digikey" H 0 0 50 0001 C CNN "SPR"
+F 7 "490-12049-1-ND" H 0 0 50 0001 C CNN "SPN"
 F 8 "" H 0 0 50 0001 C CNN "SPURL"
 	1    9750 3150

Commit message: Complete BOM. all resistors now 0402
Parts:
- U4: SPN (none) -> SC189ZSKCT-ND; SPR (none) -> Digikey
- U5: SPN (none) -> SC189ASKCT-ND; SPR (none) -> Digikey
- U6: SPN (none) -> SC189CSKCT-ND; SPR (none) -> Digikey
- U7: SPN (none) -> SC189LSKCT-ND; SPR (none) -> Digikey
