File: SD_USB.sch (KiCad schematic (older format))
At the start: 42 parts, among them CON2 AVR-JTAG-10, IC1 CyUSB30xx-BZX, J5 USB 3.0 Recept., J6 Micro_SD_Card_Det, Y1 19.2MHz

Commit message: added Zynq7020 and listed all tasks outstanding
Parts:
- removed C66, C69: 12pF, Capacitors_SMD:C_0402, symbol C_Small
- removed C67, C68: .1uF, Capacitors_SMD:C_0603, symbol C_Small
- removed IC1: CyUSB30xx-BZX, DFTcustom:BGA121_08mm, symbol CyUSB30xx-BZX
- removed J5: USB 3.0 Recept., DFTcustom:AMPHENOL_GSB3211311WEU, symbol GSB3211311WEU
- removed R29, R32, R35, R37, R38: 10k, Resistors_SMD:R_0402, symbol R_Small
- removed R36: 1k, Resistors_SMD:R_0402, symbol R_Small
- removed R57: 49.9k, Resistors_SMD:R_0402, symbol R_Small
- removed R58: 6.04k 1%, Resistors_SMD:R_0402, symbol R
- removed R59: 200 1%, Resistors_SMD:R_0402, symbol R
- removed R78, R79, R80, R81, R82: 22, Resistors_SMD:R_0402, symbol R
- removed R83: 470k, Resistors_SMD:R_0402, symbol R_Small
- removed Y1: 19.2MHz, DFTcustom:FA-20HS, symbol Crystal_Small_4pad
- added C55, C56, C57: .1uF, Capacitors_SMD:C_0603, symbol DFTBoard-rescue:C_Small-
- added R11: 4.7k, Resistors_SMD:R_0402, symbol DFTBoard-rescue:R-
- added U6: xc7z020clg400-, symbol DFTBoard-rescue:xc7z020clg400-
- added U8: TXS02612RTWR, TI:RTW, symbol TexasInstruments:TXS02612RTWR
- CON2: symbol AVR-JTAG-10 -> DFTBoard-rescue:AVR-JTAG-10-
- D1, D2, D3: renamed from D?; symbol LED -> DFTBoard-rescue:LED-
- J5: renamed from J?; symbol USB_A -> DFTBoard-rescue:USB_A-
- J6: symbol Micro_SD_Card_Det -> DFTBoard-rescue:Micro_SD_Card_Det-
- NCP1: renamed from NCP?; symbol NCP361 -> DFTBoard-rescue:NCP361-
- Q1, Q2, Q3: renamed from Q?; symbol IRLML2502 -> DFTBoard-rescue:IRLML2502-
- R10: renamed from R62; symbol R -> DFTBoard-rescue:R-
- R12: renamed from R?; symbol R -> DFTBoard-rescue:R-
- R13, R14, R15, R16, R17, R18: renamed from R?; symbol R_Small -> DFTBoard-rescue:R_Small-
- R9: renamed from R61; symbol R -> DFTBoard-rescue:R-
- U5: renamed from U?; symbol xc7z020clg400 -> DFTBoard-rescue:xc7z020clg400-
Connections:
- net labels added: RF2_IRQ, SD33_CLK, SD33_CMD, SD33_D0, SD33_D1, SD33_D2, SD33_D3, SD_CD, SD_CLK, SD_CMD, SD_D0, SD_D1, SD_D2, SD_D3, STATLED_3
- net labels removed: CONFIG_CSI, CONFIG_INIT, CONFIG_PROGRAM, CONFIG_RW, CVDDQ, FXD_N, FXD_P, RUSB2, RUSB3, SCLK, SCLKT, SCMD, SCMDT, SD0, SD0T, SD1, SD1T, SD2, SD2T, SD3, SD3T, SINS, SPIUSB_GPX, SPIUSB_INT, SPIUSB_SS, SSRX_N, SSRX_P, SSTXAC_N, SSTXAC_P, SSTX_N, SSTX_P, XN, XP, nRESET
- wire segments 90 -> 64
- no-connect marks 33 -> 28
Other:
- note added: "<- Voltage translation\nFollowing the example of Zedboard and Arty Z7"
- note added: "TODO:\nRemove 3.3V devices from 1.8V interface\nOr change this to 3.3V interface\n"
- note added: "TODO:\nUSB PHY"
- note removed: "000 => 19.2MHz crystal"
- note removed: "ID Resistors for USB 2 and 3"
- note removed: "SSTX SWAPPED ON PURPOSE"
- moved on the sheet: CON2, D1, D2, D3, J5, J6, NCP1, Q1, Q2, Q3, R10, R12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

Commit message: passes ERC, about to update footprints to v5 references
Parts:
- removed C55, C56, C57: .1uF, Capacitors_SMD:C_0603, symbol DFTBoard-rescue:C_Small-
- removed CON2: AVR-JTAG-10, DFTcustom:XilinxJTAG, symbol DFTBoard-rescue:AVR-JTAG-10-
- removed D1, D2: BLUE LED, LEDs:LED_0603, symbol DFTBoard-rescue:LED-
- removed NCP1: NCP361, DFTcustom:TSOP-5, symbol DFTBoard-rescue:NCP361-
- removed Q1, Q2, Q3: IRLML2502, TO_SOT_Packages_SMD:SOT-23, symbol DFTBoard-rescue:IRLML2502-
- removed R11: 4.7k, Resistors_SMD:R_0402, symbol DFTBoard-rescue:R-
- removed R12: 20k, Resistors_SMD:R_0402, symbol DFTBoard-rescue:R-
- removed R13, R14, R15: 1k, Resistors_SMD:R_0402, symbol DFTBoard-rescue:R_Small-
- removed R16, R17, R18: 150, Resistors_SMD:R_0402, symbol DFTBoard-rescue:R_Small-
- removed U8: TXS02612RTWR, TI:RTW, symbol TexasInstruments:TXS02612RTWR
- added C63, C64, C74, C88: .47uF, Capacitors_SMD:C_0603, symbol DFTBoard-rescue:C_Small-
- added C65, C66, C83: 4.7uF, Capacitors_SMD:C_0603, symbol DFTBoard-rescue:C_Small-
- added C67, C68, C78, C79: 100uF, Capacitors_SMD:C_1210, symbol DFTBoard-rescue:C_Small-
- added C69, C80: 2.2uF, Capacitors_SMD:C_0402, symbol DFTBoard-rescue:C
- added C70, C73, C75, C76, C77, C81, C82, C84, C87: .1uF, Capacitors_SMD:C_0603, symbol DFTBoard-rescue:C
- added C71, C72, C85, C86: 18pF, Capacitor_SMD:C_0402_1005Metric, symbol Device:C_Small
- added J8: USB_B, Connector_USB:USB_B_Amphenol_MUSB-D511_Vertical_Rugged, symbol Connector:USB_B
- added R21, R22, R23, R24, R25, R26, R27: 20k, symbol DFTBoard-rescue:R_Small
- added R30, R34, R37: 10k, Resistors_SMD:R_0402, symbol DFTBoard-rescue:R
- added R31: 47, symbol Device:R_Small
- added R32: 150, Resistors_SMD:R_0402, symbol DFTBoard-rescue:R_Small-
- added R33: 47k, symbol Device:R_Small
- added R35, R38: 1M, Resistor_SMD:R_0402_1005Metric, symbol Device:R_Small
- added R36, R39: 8.06k 1%, Resistor_SMD:R_0402_1005Metric, symbol Device:R
- added U10, U8: USB3320, Microchip:32QFN-3304-5x5B, symbol Microchip:USB3320
- added U7: S25FL256SAGNFI001, symbol parts:S25FL256SAGNFI001
- added U9: MIC2025-1YMM, Crystal:Crystal_HC35-U, symbol Micrel:MIC2025-1YMM
- added Y1, Y2: Crystal, Crystal:Crystal_HC35-U, symbol Device:Crystal
- U5: footprint (none) -> Package_BGA:BGA-400_21.0x21.0mm_Layout20x20_P1.0mm
- U5: renamed from U6; value xc7z020clg400- -> xc7z020clg400; footprint (none) -> Package_BGA:BGA-400_21.0x21.0mm_Layout20x20_P1.0mm
- renumbered J5 to J7, R9 to R28, R10 to R29
Connections:
- net labels added: BOOTSPI_CS, BOOTSPI_DQ0_BMODE3, BOOTSPI_DQ0_MODE3, BOOTSPI_DQ1_BMODE1, BOOTSPI_DQ1_MODE1, BOOTSPI_DQ2_BMODE2, BOOTSPI_DQ2_MODE2, BOOTSPI_DQ3_BMODE0, BOOTSPI_DQ3_MODE0, BOOTSPI_SCK_BMODE4, BOOTSPI_SCK_MODE4, I2C3v3_SCLK, I2C3v3_SDIN, SPI33_CLK, SPI33_MISO, SPI33_MOSI, SPI33_SS, UART33_RX, UART33_TX, USB0_CLK, USB0_D0, USB0_D1, USB0_D2, USB0_D3, USB0_D4, USB0_D5, USB0_D6, USB0_D7, USB0_RST, USB0_dir, USB0_nxt, USB0_stp, USB1_CLK, USB1_D0, USB1_D1, USB1_D2, USB1_D3, USB1_D4, USB1_D5, USB1_D6, USB1_D7, USB1_RST, USB1_dir, USB1_nxt, USB1_stp, USBD_D_N, USBD_D_P, USBD_VBUS, USBH_CPEN, USBH_D_N, USBH_D_P, USBH_FLAG_LED, USBH_VBUS, VMODE0, VMODE1
- net labels removed: FX_TCK, FX_TDI, FX_TDO, FX_TMS, FX_nTRST, I2C_SCLK, I2C_SDIN, JD_HOUT, JD_IN, JD_LOUT, JD_ROUT, SD33_CLK, SD33_CMD, SD33_D0, SD33_D1, SD33_D2, SD33_D3, SLED0_D, SLED0_G, SLED0_R, SLED1_D, SLED1_G, SLED1_R, SLED2_D, SLED2_G, SLED2_R, SPIUSB_D_N, SPIUSB_D_P, SPIUSB_VBUS, SPI_CLK, SPI_MISO, SPI_MOSI, STATLED_0, STATLED_1, STATLED_2, STATLED_3, TLV_RST#
- wire segments 64 -> 149
- no-connect marks 28 -> 9
Other:
- note added: "Active High En"
- note added: "Both Banks 3v3"
- note added: "Device USB 1"
- note added: "Fixed Host Mode"
- note added: "Host USB 0"
- note added: "PLLs Enabled, \nJTAG Cascade,\nQSPI Boot"
- note added: "RGMII Ref, \nSafe to Float"
- note removed: "<- Voltage translation\nFollowing the example of Zedboard and Arty Z7"
- note removed: "TODO:\nRemove 3.3V devices from 1.8V interface\nOr change this to 3.3V interface\n"
- note removed: "TODO:\nUSB PHY"
- moved on the sheet: J6, J7, R28, R29

Commit message: still works, miraculously
Parts:
- C63, C64, C65, C66, C74, C83, C88: footprint Capacitors_SMD:C_0603 -> Capacitor_SMD:C_0603_1608Metric; symbol DFTBoard-rescue:C_Small- -> Device:C_Small
- C67, C68, C78, C79: symbol DFTBoard-rescue:C_Small- -> Device:C_Small
- C69, C80: symbol DFTBoard-rescue:C -> Device:C
- C70, C73, C75, C76, C77, C81, C82, C84, C87: footprint Capacitors_SMD:C_0603 -> Capacitor_SMD:C_0603_1608Metric; symbol DFTBoard-rescue:C -> Device:C
- R21, R22, R23, R24, R25, R26, R27: symbol DFTBoard-rescue:R_Small -> Device:R_Small
- R28, R29: symbol DFTBoard-rescue:R- -> Device:R
- R30, R34, R37: symbol DFTBoard-rescue:R -> Device:R
- R32: symbol DFTBoard-rescue:R_Small- -> Device:R_Small
Connections:
- net +1.8V renamed +1V8

Commit message: random updates
Parts:
- R28, R29, R30, R32, R34, R37: footprint Resistors_SMD:R_0402 -> Resistor_SMD:R_0402_1005Metric
Changed lines of the file:
@@
 F 0 "R28" V 880 2050 50  0000 C CNN
 F 1 "4.7k" V 800 2050 50  0000 C CNN
-F 2 "Resistors_SMD:R_0402" V 730 2050 50  0001 C CNN
+F 2 "Resistor_SMD:R_0402_1005Metric" V 730 2050 50  0001 C CNN
 F 3 "" H 800 2050 50  0001 C CNN
 F 4 "Yageo" H -1550 -5250 50  0001 C CNN "MFR"
@@
 F 0 "R29" V 1080 2050 50  0000 C CNN
 F 1 "4.7k" V 1000 2050 50  0000 C CNN
-F 2 "Resistors_SMD:R_0402" V 930 2050 50  0001 C CNN
+F 2 "Resistor_SMD:R_0402_1005Metric" V 930 2050 50  0001 C CNN
 F 3 "" H 1000 2050 50  0001 C CNN
 F 4 "Yageo" H -1550 -5350 50  0001 C CNN "MFR"
@@
 F 0 "R34" V 3950 2550 50  0000 C CNN
 F 1 "10k" V 4050 2550 50  0000 C CNN
-F 2 "Resistors_SMD:R_0402" V 3980 2550 50  0001 C CNN
+F 2 "Resistor_SMD:R_0402_1005Metric" V 3980 2550 50  0001 C CNN
 F 3 "" H 4050 2550 50  0001 C CNN
 F 4 "Yageo" H -2050 -200 50  0001 C CNN "MFR"
@@
 F 0 "R32" H 3880 1370 50  0000 L CNN
 F 1 "150" H 3880 1310 50  0000 L CNN
-F 2 "Resistors_SMD:R_0402" H 3850 1350 50  0001 C CNN
+F 2 "Resistor_SMD:R_0402_1005Metric" H 3850 1350 50  0001 C CNN
 F 3 "" H 3850 1350 50  0001 C CNN
 F 4 "Yageo" H 1800 -3000 50  0001 C CNN "MFR"
@@
 F 0 "R37" V 8000 1400 50  0000 C CNN
 F 1 "10k" V 8100 1400 50  0000 C CNN
-F 2 "Resistors_SMD:R_0402" V 8030 1400 50  0001 C CNN
+F 2 "Resistor_SMD:R_0402_1005Metric" V 8030 1400 50  0001 C CNN
 F 3 "" H 8100 1400 50  0001 C CNN
 F 4 "Yageo" H 2000 -1350 50  0001 C CNN "MFR"
@@
 F 0 "R30" V 1600 7200 50  0000 C CNN
 F 1 "10k" V 1700 7200 50  0000 C CNN
-F 2 "Resistors_SMD:R_0402" V 1630 7200 50  0001 C CNN
+F 2 "Resistor_SMD:R_0402_1005Metric" V 1630 7200 50  0001 C CNN
 F 3 "" H 1700 7200 50  0001 C CNN
 F 4 "Yageo" H -4400 4450 50  0001 C CNN "MFR"
