File: DDR3.sch (KiCad schematic (older format))
At the start: 20 parts, among them U11 W9751G6KB

Commit message: added Zynq7020 and listed all tasks outstanding
Parts:
- added C64, C70: 10uF, Capacitors_SMD:C_0603, symbol DFTBoard-rescue:C_Small-
- added C68, C69, C72, C74, C77, C78: .1uF, Capacitors_SMD:C_0603, symbol DFTBoard-rescue:C_Small-
- added R25, R26: 10k, Resistors_SMD:R_0402, symbol DFTBoard-rescue:R_Small-
- added U12: W9751G6KB, DFTcustom:WBGA-84, symbol DFTBoard-rescue:W9751G6KB-
- C63: renamed from C134; symbol C_Small -> DFTBoard-rescue:C_Small-
- C65: renamed from C123; symbol C_Small -> DFTBoard-rescue:C_Small-
- C66: renamed from C125; symbol C_Small -> DFTBoard-rescue:C_Small-
- C67: renamed from C135; symbol C_Small -> DFTBoard-rescue:C_Small-
- C71: renamed from C136; symbol C_Small -> DFTBoard-rescue:C_Small-
- C73: renamed from C137; symbol C_Small -> DFTBoard-rescue:C_Small-
- C75: renamed from C124; symbol C_Small -> DFTBoard-rescue:C_Small-
- C76: renamed from C126; symbol C_Small -> DFTBoard-rescue:C_Small-
- C79: renamed from C127; symbol C_Small -> DFTBoard-rescue:C_Small-
- C80: renamed from C128; symbol C_Small -> DFTBoard-rescue:C_Small-
- C81: renamed from C129; symbol C_Small -> DFTBoard-rescue:C_Small-
- C82: renamed from C130; symbol C_Small -> DFTBoard-rescue:C_Small-
- C83: renamed from C131; symbol C_Small -> DFTBoard-rescue:C_Small-
- C84: renamed from C132; symbol C_Small -> DFTBoard-rescue:C_Small-
- C85: renamed from C133; symbol C_Small -> DFTBoard-rescue:C_Small-
- R23: renamed from R75; symbol R_Small -> DFTBoard-rescue:R_Small-
- R24: renamed from R76; symbol R_Small -> DFTBoard-rescue:R_Small-
- R27: renamed from R77; symbol R -> DFTBoard-rescue:R-
- U11: symbol W9751G6KB -> DFTBoard-rescue:W9751G6KB-
- U5: renamed from U?; symbol xc7z020clg400 -> DFTBoard-rescue:xc7z020clg400-
Connections:
- net labels added: DDR3_A0, DDR3_A1, DDR3_A10, DDR3_A11, DDR3_A12, DDR3_A2, DDR3_A3, DDR3_A4, DDR3_A5, DDR3_A6, DDR3_A7, DDR3_A8, DDR3_A9, DDR3_BA0, DDR3_BA1, DDR3_CAS#, DDR3_CKE, DDR3_CK_N, DDR3_CK_P, DDR3_CS, DDR3_DM0, DDR3_DM1, DDR3_DM2, DDR3_DM3, DDR3_DQ0, DDR3_DQ1, DDR3_DQ10, DDR3_DQ11, DDR3_DQ12, DDR3_DQ13, DDR3_DQ14, DDR3_DQ15, DDR3_DQ16, DDR3_DQ17, DDR3_DQ18, DDR3_DQ19, DDR3_DQ2, DDR3_DQ20, DDR3_DQ21, DDR3_DQ22, DDR3_DQ23, DDR3_DQ24, DDR3_DQ25, DDR3_DQ26, DDR3_DQ27, DDR3_DQ28, DDR3_DQ29, DDR3_DQ3, DDR3_DQ30, DDR3_DQ31, DDR3_DQ4, DDR3_DQ5, DDR3_DQ6, DDR3_DQ7, DDR3_DQ8, DDR3_DQ9, DDR3_DQS0_N, DDR3_DQS0_P, DDR3_DQS1_N, DDR3_DQS1_P, DDR3_DQS2_N, DDR3_DQS2_P, DDR3_DQS3_N, DDR3_DQS3_P, DDR3_ODT, DDR3_RAS#, DDR3_WE#
- net labels removed: RAM_A0, RAM_A1, RAM_A10, RAM_A11, RAM_A12, RAM_A2, RAM_A3, RAM_A4, RAM_A5, RAM_A6, RAM_A7, RAM_A8, RAM_A9, RAM_BA0, RAM_BA1, RAM_CAS#, RAM_CKE, RAM_CK_N, RAM_CK_P, RAM_DQ0, RAM_DQ1, RAM_DQ10, RAM_DQ11, RAM_DQ12, RAM_DQ13, RAM_DQ14, RAM_DQ15, RAM_DQ2, RAM_DQ3, RAM_DQ4, RAM_DQ5, RAM_DQ6, RAM_DQ7, RAM_DQ8, RAM_DQ9, RAM_LDQS_N, RAM_LDQS_P, RAM_ODT, RAM_RAS#, RAM_UDQS_N, RAM_UDQS_P, RAM_WE#
- wire segments 73 -> 232
- no-connect marks 1 -> 5
Other:
- note added: "TODO: \nTerminations as described in UG933\nand shown in ZC702 schematic"
- moved on the sheet: C63, C65, C66, C67, C71, C73, C75, C76, C79, C80, C81, C82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

Commit message: passes ERC, about to update footprints to v5 references
Parts:
- removed C63, C64, C67, C70: 10uF, Capacitors_SMD:C_0603, symbol DFTBoard-rescue:C_Small-
- removed C68, C69, C71, C72, C73, C74, C77, C78: .1uF, Capacitors_SMD:C_0603, symbol DFTBoard-rescue:C_Small-
- removed C79: 47uF, Capacitors_SMD:C_1210, symbol DFTBoard-rescue:C_Small-
- removed C80: 4.7uF, Capacitors_SMD:C_0603, symbol DFTBoard-rescue:C_Small-
- removed R24, R25, R26: 10k, Resistors_SMD:R_0402, symbol DFTBoard-rescue:R_Small-
- removed U11, U12: W9751G6KB, DFTcustom:WBGA-84, symbol DFTBoard-rescue:W9751G6KB-
- added C105, C106, C93, C98: .01uF, Capacitors_SMD:C_0603, symbol DFTBoard-rescue:C_Small-
- added C99: 100uF, Capacitors_SMD:C_1210, symbol DFTBoard-rescue:C_Small-
- added R46, R49: 240 1%, Resistor_SMD:R_0402_1005Metric, symbol Device:R
- added R48: 10k 1%, Resistors_SMD:R_0402, symbol DFTBoard-rescue:R_Small-
- added R51, R52, R53, R54, R55, R56, R57, R58, R59, R60, R61, R62, R63, R64, R65, R66, R67, R68, R69, R70, R71, R72, R73: 40.2 1%, Resistor_SMD:R_0201_0603Metric, symbol DFTBoard-rescue:R_Small
- added R74: 4.7k, Resistor_SMD:R_0402_1005Metric, symbol DFTBoard-rescue:R_Small
- added R75, R76: 80.6, Resistor_SMD:R_0402_1005Metric, symbol Device:R
- added U15, U16: MT41K256M16HA-125_E, DFTcustom:FBGA-96-DDR3-SDRAM, symbol MT41K256M16HA-125_E:MT41K256M16HA-125_E
- R47: renamed from R23; value 10k -> 10k 1%; MPN RC0402FR-0710KL -> (none); SPN 311-10.0KLRTR-ND -> (none)
- U8: renamed from U5; footprint (none) -> Package_BGA:BGA-400_21.0x21.0mm_Layout20x20_P1.0mm
- renumbered C81 to C100, C82 to C101, C83 to C102, C84 to C103, C85 to C104, C65 to C94, C66 to C95, C75 to C96, C76 to C97, R27 to R50
Connections:
- net DDR3_A0: now also R51.1, U15.N3 (A0), U16.N3 (A0)
- net DDR3_A1: now also R52.1, U15.P7 (A1), U16.P7 (A1)
- net DDR3_A10: now also R61.1, U15.L7 (A10/AP), U16.L7 (A10/AP)
- net DDR3_A11: now also R62.1, U15.R7 (A11), U16.R7 (A11)
- net DDR3_A12: now also R63.1, U15.N7 (A12/!BC), U16.N7 (A12/!BC)
- net DDR3_A2: now also R53.1, U15.P3 (A2), U16.P3 (A2)
- net DDR3_A3: now also R54.1, U15.N2 (A3), U16.N2 (A3)
- net DDR3_A4: now also R55.1, U15.P8 (A4), U16.P8 (A4)
- net DDR3_A5: now also R56.1, U15.P2 (A5), U16.P2 (A5)
- net DDR3_A6: now also R57.1, U15.R8 (A6), U16.R8 (A6)
- net DDR3_A7: now also R58.1, U15.R2 (A7), U16.R2 (A7)
- net DDR3_A8: now also R59.1, U15.T8 (A8), U16.T8 (A8)
- net DDR3_A9: now also R60.1, U15.R3 (A9), U16.R3 (A9)
- net DDR3_BA0: now also R66.1, U15.M2 (BA0), U16.M2 (BA0)
- net DDR3_BA1: now also R67.1, U15.N8 (BA1), U16.N8 (BA1)
- net DDR3_CAS#: now also R70.1, U15.K3 (~CAS~), U16.K3 (~CAS~)
- net DDR3_CKE: now also U15.K9 (CKE), U16.K9 (CKE)
- net DDR3_CK_N: now also U15.K7 (~CK~), U16.K7 (~CK~)
- net DDR3_CK_P: now also U15.J7 (CK), U16.J7 (CK)
- net DDR3_DM0: now also U16.E7 (LDM)
- net DDR3_DM1: now also U16.D3 (UDM)
- net DDR3_DM2: now also U15.E7 (LDM)
- net DDR3_DM3: now also U15.D3 (UDM)
- net DDR3_DQ0: now also U16.E3 (DQ0)
- net DDR3_DQ1: now also U16.F7 (DQ1)
- net DDR3_DQ10: now also U16.C8 (DQ10)
- net DDR3_DQ11: now also U16.C2 (DQ11)
- net DDR3_DQ12: now also U16.A7 (DQ12)
- net DDR3_DQ13: now also U16.A2 (DQ13)
- net DDR3_DQ14: now also U16.B8 (DQ14)
- net DDR3_DQ15: now also U16.A3 (DQ15)
- net DDR3_DQ16: now also U15.E3 (DQ0)
- net DDR3_DQ17: now also U15.F7 (DQ1)
- net DDR3_DQ18: now also U15.F2 (DQ2)
- net DDR3_DQ19: now also U15.F8 (DQ3)
- net DDR3_DQ2: now also U16.F2 (DQ2)
- net DDR3_DQ20: now also U15.H3 (DQ4)
- net DDR3_DQ21: now also U15.H8 (DQ5)
- net DDR3_DQ22: now also U15.G2 (DQ6)
- net DDR3_DQ23: now also U15.H7 (DQ7)
- net DDR3_DQ24: now also U15.D7 (DQ8)
- net DDR3_DQ25: now also U15.C3 (DQ9)
- net DDR3_DQ26: now also U15.C8 (DQ10)
- net DDR3_DQ27: now also U15.C2 (DQ11)
- net DDR3_DQ28: now also U15.A7 (DQ12)
- net DDR3_DQ29: now also U15.A2 (DQ13)
- net DDR3_DQ3: now also U16.F8 (DQ3)
- net DDR3_DQ30: now also U15.B8 (DQ14)
- net DDR3_DQ31: now also U15.A3 (DQ15)
- net DDR3_DQ4: now also U16.H3 (DQ4)
- net DDR3_DQ5: now also U16.H8 (DQ5)
- net DDR3_DQ6: now also U16.G2 (DQ6)
- net DDR3_DQ7: now also U16.H7 (DQ7)
- net DDR3_DQ8: now also U16.D7 (DQ8)
- net DDR3_DQ9: now also U16.C3 (DQ9)
- net DDR3_DQS0_N: now also U16.G3 (~LDQS~)
- net DDR3_DQS0_P: now also U16.F3 (LDQS)
- net DDR3_DQS1_N: now also U16.B7 (~UDQS~)
- net DDR3_DQS1_P: now also U16.C7 (UDQS)
- net DDR3_DQS2_N: now also U15.G3 (~LDQS~)
- net DDR3_DQS2_P: now also U15.F3 (LDQS)
- net DDR3_DQS3_N: now also U15.B7 (~UDQS~)
- net DDR3_DQS3_P: now also U15.C7 (UDQS)
- net DDR3_ODT: now also R72.1, U15.K1 (ODT), U16.K1 (ODT)
- net DDR3_RAS#: now also R69.1, U15.J3 (~RAS~), U16.J3 (~RAS~)
- net DDR3_WE#: now also R71.1, U15.L3 (~WE~), U16.L3 (~WE~)
- net GND: now also C105.2, C106.2, C93.2, C98.2, C99.2, R46.2, R48.2, R49.2, R74.2, R76.2, U15.A9 (VSS), U15.B1 (VSSQ), U15.B3 (VSS), U15.B9 (VSSQ), U15.D1 (VSSQ), U15.D8 (VSSQ), U15.E1 (VSS), U15.E2 (VSSQ), U15.E8 (VSSQ), U15.F9 (VSSQ), U15.G1 (VSSQ), U15.G8 (VSS), U15.G9 (VSSQ), U15.J2 (VSS), U15.J8 (VSS), U15.M1 (VSS), U15.M9 (VSS), U15.P1 (VSS), U15.P9 (VSS), U15.T1 (VSS), U15.T9 (VSS), U16.A9 (VSS), U16.B1 (VSSQ), U16.B3 (VSS), U16.B9 (VSSQ), U16.D1 (VSSQ), U16.D8 (VSSQ), U16.E1 (VSS), U16.E2 (VSSQ), U16.E8 (VSSQ), U16.F9 (VSSQ), U16.G1 (VSSQ), U16.G8 (VSS), U16.G9 (VSSQ), U16.J2 (VSS), U16.J8 (VSS), U16.M1 (VSS), U16.M9 (VSS), U16.P1 (VSS), U16.P9 (VSS), U16.T1 (VSS), U16.T9 (VSS)
- net VREF: now also U8.H6 (PS_DDR_VREF0_502), U8.P6 (PS_DDR_VREF1_502), C105.1, C106.1, C93.1, C98.1, R48.1, U15.H1 (VREFDQ), U15.M8 (VREFCA), U16.H1 (VREFDQ), U16.M8 (VREFCA)
- net DDR3_DRST#: now reaches U8.B4 (PS_DDR_DRST_B_502)
- net DDR3_DRST#: now also R74.1, U15.T2 (~RESET~), U16.T2 (~RESET~)
- net DDR3_A13: now reaches U8.D4 (PS_DDR_A13_502)
- net DDR3_A13: now also R64.1, U15.T3 (A13), U16.T3 (A13)
- net DDR3_A14: now reaches U8.F4 (PS_DDR_A14_502)
- net DDR3_A14: now also R65.1, U15.T7 (A14), U16.T7 (A14)
- net at U8.G5 (PS_DDR_VRN_502): now also R75.1
- net at U8.H5 (PS_DDR_VRP_502): now also R76.1
- net DDR3_BA2: now reaches U8.J5 (PS_DDR_BA2_502)
- net DDR3_BA2: now also R68.1, U15.M3 (BA2), U16.M3 (BA2)
- net +1.8V renamed +1V35
- net +1V35: now also C99.1, R51.2, R52.2, R53.2, R54.2, R55.2, R56.2, R57.2, R58.2, R59.2, R60.2, R61.2, R62.2, R63.2, R64.2, R65.2, R66.2, R67.2, R68.2, R69.2, R70.2, R71.2, R72.2, R73.2, R75.2, U15.A1 (VDDQ), U15.A8 (VDDQ), U15.B2 (VDD), U15.C1 (VDDQ), U15.C9 (VDDQ), U15.D2 (VDDQ), U15.D9 (VDD), U15.E9 (VDDQ), U15.F1 (VDDQ), U15.G7 (VDD), U15.H2 (VDDQ), U15.H9 (VDDQ), U15.K2 (VDD), U15.K8 (VDD), U15.N1 (VDD), U15.N9 (VDD), U15.R1 (VDD), U15.R9 (VDD), U16.A1 (VDDQ), U16.A8 (VDDQ), U16.B2 (VDD), U16.C1 (VDDQ), U16.C9 (VDDQ), U16.D2 (VDDQ), U16.D9 (VDD), U16.E9 (VDDQ), U16.F1 (VDDQ), U16.G7 (VDD), U16.H2 (VDDQ), U16.H9 (VDDQ), U16.K2 (VDD), U16.K8 (VDD), U16.N1 (VDD), U16.N9 (VDD), U16.R1 (VDD), U16.R9 (VDD)
- net DDR3_CS renamed DDR3_CS#
- net DDR3_CS#: now also R73.1, U15.L2 (~CS~), U16.L2 (~CS~)
- new net: R49.1, U16.L8 (ZQ)
- new net: R46.1, U15.L8 (ZQ)
- no-connect marks 5 -> 0
Other:
- note added: "DDR3L trace impedance:\n40ohm differential\n80ohm single"
- note added: "Pinout identical to TW \n96-ball FBGA variant\n"
- note added: "RECOMMENDED: Fly-by and \npoint-to-point routing is\nrecommended for optimal \nmemory performance"
- note added: "Terminations as described in UG933\nand shown in ZC702 schematic"
- note removed: "TODO: \nTerminations as described in UG933\nand shown in ZC702 schematic"
- moved on the sheet: C100, C101, C102, C103, C104, C94, C95, C96, C97, R47, R50, U8G

Commit message: replacing rescue components foreal
Parts:
- U8: footprint Package_BGA:BGA-400_21.0x21.0mm_Layout20x20_P1.0mm -> DFTcustom:BGA400_0.8p_17mmx17mm
Changed lines of the file:
@@
 F 0 "U8" H 10350 700 60  0000 L CNN
 F 1 "xc7z020clg400" H 10350 600 60  0000 L CNN
-F 2 "Package_BGA:BGA-400_21.0x21.0mm_Layout20x20_P1.0mm" H 10150 450 60  0001 C CNN
+F 2 "DFTcustom:BGA400_0.8p_17mmx17mm" H 10150 450 60  0001 C CNN
 F 3 "" H 10150 450 60  0001 C CNN
 	7    10150 450

Commit message: still works, miraculously
Parts:
- C100, C101, C102, C103, C104, C105, C106, C93, C94, C95, C96, C97, C98: footprint Capacitors_SMD:C_0603 -> Capacitor_SMD:C_0603_1608Metric; symbol DFTBoard-rescue:C_Small- -> Device:C_Small
- C99: footprint Capacitors_SMD:C_1210 -> Capacitor_SMD:C_1210_3225Metric; symbol DFTBoard-rescue:C_Small- -> Device:C_Small
- R47, R48: symbol DFTBoard-rescue:R_Small- -> Device:R_Small
- R50: symbol DFTBoard-rescue:R- -> Device:R
- R51, R52, R53, R54, R55, R56, R57, R58, R59, R60, R61, R62, R63, R64, R65, R66, R67, R68, R69, R70, R71, R72, R73, R74: symbol DFTBoard-rescue:R_Small -> Device:R_Small
Changed lines of the file:
@@
 $EndDescr
 $Comp
-L DFTBoard-rescue:R_Small- R47
+L Device:R_Small R47
 U 1 1 58829D91
 P 2800 6850
@@
 $EndComp
 $Comp
-L DFTBoard-rescue:GND- #PWR0154
+L power:GND #PWR0154
 U 1 1 58829F20
 P 2800 7600
@@
 $EndComp
 $Comp
-L DFTBoard-rescue:C_Small- C94
+L Device:C_Small C94
 U 1 1 5882A26A
 P 2500 6850
 F 0 "C94" H 2510 6920 50  0000 L CNN
 F 1 ".1uF" H 2510 6770 50  0000 L CNN
-F 2 "Capacitors_SMD:C_0603" H 2500 6850 50  0001 C CNN
+F 2 "Capacitor_SMD:C_0603_1608Metric" H 2500 6850 50  0001 C CNN
 F 3 "" H 2500 6850 50  0001 C CNN
 F 4 "Murata" H 1500 2300 50  0001 C CNN "MFR"
@@
 $EndComp
 $Comp
-L DFTBoard-rescue:C_Small- C95
+L Device:C_Small C95
 U 1 1 5882A2B4
 P 2500 7350
 F 0 "C95" H 2510 7420 50  0000 L CNN
 F 1 ".1uF" H 2510 7270 50  0000 L CNN
-F 2 "Capacitors_SMD:C_0603" H 2500 7350 50  0001 C CNN
+F 2 "Capacitor_SMD:C_0603_1608Metric" H 2500 7350 50  0001 C CNN
 F 3 "" H 2500 7350 50  0001 C CNN
 F 4 "Murata" H 1500 2300 50  0001 C CNN "MFR"
@@
 $EndComp
 $Comp
-L DFTBoard-rescue:C_Small- C96
+L Device:C_Small C96
 U 1 1 5882A2F8
 P 3100 6850
 F 0 "C96" H 3110 6920 50  0000 L CNN
 F 1 ".1uF" H 3110 6770 50  0000 L CNN
-F 2 "Capacitors_SMD:C_0603" H 3100 6850 50  0001 C CNN
+F 2 "Capacitor_SMD:C_0603_1608Metric" H 3100 6850 50  0001 C CNN
 F 3 "" H 3100 6850 50  0001 C CNN
 F 4 "Murata" H 1500 2300 50  0001 C CNN "MFR"
@@
 $EndComp
 $Comp
-L DFTBoard-rescue:C_Small- C97
+L Device:C_Small C97
 U 1 1 5882A33B
 P 3100 7350
 F 0 "C97" H 3110 7420 50  0000 L CNN
 F 1 ".1uF" H 3110 7270 50  0000 L CNN
-F 2 "Capacitors_SMD:C_0603" H 3100 7350 50  0001 C CNN
+F 2 "Capacitor_SMD:C_0603_1608Metric" H 3100 7350 50  0001 C CNN
 F 3 "" H 3100 7350 50  0001 C CNN
 F 4 "Murata" H 1500 2300 50  0001 C CNN "MFR"
@@
 $EndComp
 $Comp
-L DFTBoard-rescue:C_Small- C100
+L Device:C_Small C100
 U 1 1 5887E429
 P 8050 6100
 F 0 "C100" H 8060 6170 50  0000 L CNN
 F 1 "4.7uF" H 8060 6020 50  0000 L CNN
-F 2 "Capacitors_SMD:C_0603" H 8050 6100 50  0001 C CNN
+F 2 "Capacitor_SMD:C_0603_1608Metric" H 8050 6100 50  0001 C CNN
 F 3 "" H 8050 6100 50  0001 C CNN
 F 4 "Murata" H 650 150 50  0001 C CNN "MFR"
@@
 $EndComp
 $Comp
-L DFTBoard-rescue:C_Small- C101
+L Device:C_Small C101
 U 1 1 5887E430
 P 8300 6100
 F 0 "C101" H 8310 6170 50  0000 L CNN
 F 1 ".47uF" H 8310 6020 50  0000 L CNN
-F 2 "Capacitors_SMD:C_0603" H 8300 6100 50  0001 C CNN
+F 2 "Capacitor_SMD:C_0603_1608Metric" H 8300 6100 50  0001 C CNN
 F 3 "" H 8300 6100 50  0001 C CNN
 F 4 "Murata" H 650 150 50  0001 C CNN "MFR"
@@
 $EndComp
 $Comp
-L DFTBoard-rescue:C_Small- C102
+L Device:C_Small C102
 U 1 1 5887E437
 P 8550 6100
 F 0 "C102" H 8560 6170 50  0000 L CNN
 F 1 ".47uF" H 8560 6020 50  0000 L CNN
-F 2 "Capacitors_SMD:C_0603" H 8550 6100 50  0001 C CNN
+F 2 "Capacitor_SMD:C_0603_1608Metric" H 8550 6100 50  0001 C CNN
 F 3 "" H 8550 6100 50  0001 C CNN
 F 4 "Murata" H 650 150 50  0001 C CNN "MFR"
@@
 $EndComp
 $Comp
-L DFTBoard-rescue:C_Small- C103
+L Device:C_Small C103
 U 1 1 5887E43E
 P 8800 6100
 F 0 "C103" H 8810 6170 50  0000 L CNN
 F 1 ".47uF" H 8810 6020 50  0000 L CNN
-F 2 "Capacitors_SMD:C_0603" H 8800 6100 50  0001 C CNN
+F 2 "Capacitor_SMD:C_0603_1608Metric" H 8800 6100 50  0001 C CNN
 F 3 "" H 8800 6100 50  0001 C CNN
 F 4 "Murata" H 650 150 50  0001 C CNN "MFR"
@@
 $EndComp
 $Comp
-L DFTBoard-rescue:C_Small- C104
+L Device:C_Small C104
 U 1 1 5887E445
 P 9050 6100
 F 0 "C104" H 9060 6170 50  0000 L CNN
 F 1 ".47uF" H 9060 6020 50  0000 L CNN
-F 2 "Capacitors_SMD:C_0603" H 9050 6100 50  0001 C CNN
+F 2 "Capacitor_SMD:C_0603_1608Metric" H 9050 6100 50  0001 C CNN
 F 3 "" H 9050 6100 50  0001 C CNN
 F 4 "Murata" H 650 150 50  0001 C CNN "MFR"
@@
 $EndComp
 $Comp
-L DFTBoard-rescue:GND- #PWR0162
+L power:GND #PWR0162
 U 1 1 5887E465
 P 8050 6400
@@
 DDR3_CK_N
 $Comp
-L DFTBoard-rescue:R- R50
+L Device:R R50
 U 1 1 5A7D1ACF
 P 5800 1050
@@
 Terminations as described in UG933\nand shown in ZC702 schematic
 $Comp
-L DFTBoard-rescue:C_Small- C?
+L Device:C_Small C?
 U 1 1 5CB10B71
 P 7800 6100
@@
 F 0 "C99" H 7810 6170 50  0000 L CNN
 F 1 "100uF" H 7810 6020 50  0000 L CNN
-F 2 "Capacitors_SMD:C_1210" H 7800 6100 50  0001 C CNN
+F 2 "Capacitor_SMD:C_1210_3225Metric" H 7800 6100 50  0001 C CNN
 F 3 "" H 7800 6100 50  0001 C CNN
 F 4 "TAIYO YUDEN" H 4300 1050 50  0001 C CNN "MFR"
@@
 	3850 5750 3850 5850
 $Comp
-L DFTBoard-rescue:GND- #PWR0155
+L power:GND #PWR0155
 U 1 1 5C8E3DDA
 P 3850 6150
@@
 DDR3_DQ0
 $Comp
-L DFTBoard-rescue:GND- #PWR0157
+L power:GND #PWR0157
 U 1 1 588278E2
 P 5550 6200
@@
 	2450 5900 2550 5900
 $Comp
-L DFTBoard-rescue:GND- #PWR0151
+L power:GND #PWR0151
 U 1 1 5C8EEF2B
 P 2550 6150
@@
 	850  5700 850  5800
 $Comp
-L DFTBoard-rescue:GND- #PWR0149
+L power:GND #PWR0149
 U 1 1 5C8FB945
 P 850 6100
@@
 VREF
 $Comp
-L DFTBoard-rescue:C_Small- C93
+L Device:C_Small C93
 U 1 1 5C964448
 P 2450 2300
 F 0 "C93" H 2460 2370 50  0000 L CNN
 F 1 ".01uF" H 2460 2220 50  0000 L CNN
-F 2 "Capacitors_SMD:C_0603" H 2450 2300 50  0001 C CNN
+F 2 "Capacitor_SMD:C_0603_1608Metric" H 2450 2300 50  0001 C CNN
 F 3 "" H 2450 2300 50  0001 C CNN
 F 4 "Murata" H 850 -2250 50  0001 C CNN "MFR"
@@
 $EndComp
 $Comp
-L DFTBoard-rescue:GND- #PWR0150
+L power:GND #PWR0150
 U 1 1 5C96467C
 P 2450 2400
@@
 $EndComp
 $Comp
-L DFTBoard-rescue:C_Small- C106
+L Device:C_Small C106
 U 1 1 5C96471D
 P 9050 7650
 F 0 "C106" H 9060 7720 50  0000 L CNN
 F 1 ".01uF" H 9060 7570 50  0000 L CNN
-F 2 "Capacitors_SMD:C_0603" H 9050 7650 50  0001 C CNN
+F 2 "Capacitor_SMD:C_0603_1608Metric" H 9050 7650 50  0001 C CNN
 F 3 "" H 9050 7650 50  0001 C CNN
 F 4 "Murata" H 7450 3100 50  0001 C CNN "MFR"
@@
 $EndComp
 $Comp
-L DFTBoard-rescue:C_Small- C105
+L Device:C_Small C105
 U 1 1 5C96492F
 P 8750 7550
 F 0 "C105" H 8760 7620 50  0000 L CNN
 F 1 ".01uF" H 8760 7470 50  0000 L CNN
-F 2 "Capacitors_SMD:C_0603" H 8750 7550 50  0001 C CNN
+F 2 "Capacitor_SMD:C_0603_1608Metric" H 8750 7550 50  0001 C CNN
 F 3 "" H 8750 7550 50  0001 C CNN
 F 4 "Murata" H 7150 3000 50  0001 C CNN "MFR"
@@
 $EndComp
 $Comp
-L DFTBoard-rescue:GND- #PWR0164
+L power:GND #PWR0164
 U 1 1 5C9719EC
 P 9050 7750
@@
 $EndComp
 $Comp
-L DFTBoard-rescue:GND- #PWR0163
+L power:GND #PWR0163
 U 1 1 5C971AD3
 P 8750 7650
@@
 $EndComp
 $Comp
-L DFTBoard-rescue:GND- #PWR0166
+L power:GND #PWR0166
 U 1 1 5C97700F
 P 9650 7750
@@
 $EndComp
 $Comp
-L DFTBoard-rescue:C_Small- C98
+L Device:C_Small C98
 U 1 1 5C97BD40
 P 5500 2300
 F 0 "C98" H 5510 2370 50  0000 L CNN
 F 1 ".01uF" H 5510 2220 50  0000 L CNN
-F 2 "Capacitors_SMD:C_0603" H 5500 2300 50  0001 C CNN
+F 2 "Capacitor_SMD:C_0603_1608Metric" H 5500 2300 50  0001 C CNN
 F 3 "" H 5500 2300 50  0001 C CNN
 F 4 "Murata" H 3900 -2250 50  0001 C CNN "MFR"
@@
 	5500 2200 5600 2200
 $Comp
-L DFTBoard-rescue:GND- #PWR0156
+L power:GND #PWR0156
 U 1 1 5C97BFA2
 P 5500 2400
@@
 $EndComp
 $Comp
-L DFTBoard-rescue:R_Small- R48
+L Device:R_Small R48
 U 1 1 5C97C3FF
 P 2800 7350
@@
 $EndComp
 $Comp
-L DFTBoard-rescue:R_Small R52
+L Device:R_Small R52
 U 1 1 5C9CB426
 P 7750 1700
@@
 DDR3_A14
 $Comp
-L DFTBoard-rescue:R_Small R51
+L Device:R_Small R51
 U 1 1 5C9EBED7
 P 7750 1600
@@
 $EndComp
 $Comp
-L DFTBoard-rescue:R_Small R54
+L Device:R_Small R54
 U 1 1 5C9EDA10
 P 7750 1900
@@
 $EndComp
 $Comp
-L DFTBoard-rescue:R_Small R53
+L Device:R_Small R53
 U 1 1 5C9EDA16
 P 7750 1800
@@
 $EndComp
 $Comp
-L DFTBoard-rescue:R_Small R56
+L Device:R_Small R56
 U 1 1 5C9EF607
 P 7750 2100
@@
 $EndComp
 $Comp
-L DFTBoard-rescue:R_Small R55
+L Device:R_Small R55
 U 1 1 5C9EF60D
 P 7750 2000
@@
 $EndComp
 $Comp
-L DFTBoard-rescue:R_Small R58
+L Device:R_Small R58
 U 1 1 5C9EF613
 P 7750 2300
@@
 $EndComp
 $Comp
-L DFTBoard-rescue:R_Small R57
+L Device:R_Small R57
 U 1 1 5C9EF619
 P 7750 2200
@@
 $EndComp
 $Comp
-L DFTBoard-rescue:R_Small R60
+L Device:R_Small R60
 U 1 1 5C9F1272
 P 7750 2500
@@
 $EndComp
 $Comp
-L DFTBoard-rescue:R_Small R59
+L Device:R_Small R59
 U 1 1 5C9F1278
 P 7750 2400
@@
 $EndComp
 $Comp
-L DFTBoard-rescue:R_Small R62
+L Device:R_Small R62
 U 1 1 5C9F127E
 P 7750 2700
@@
 $EndComp
 $Comp
-L DFTBoard-rescue:R_Small R61
+L Device:R_Small R61
 U 1 1 5C9F1284
 P 7750 2600
@@
 $EndComp
 $Comp
-L DFTBoard-rescue:R_Small R64
+L Device:R_Small R64
 U 1 1 5C9F128A
 P 7750 2900
@@
 $EndComp
 $Comp
-L DFTBoard-rescue:R_Small R63
+L Device:R_Small R63
 U 1 1 5C9F1290
 P 7750 2800
@@
 $EndComp
 $Comp
-L DFTBoard-rescue:R_Small R66
+L Device:R_Small R66
 U 1 1 5C9F1296
 P 7750 3200
@@
 $EndComp
 $Comp
-L DFTBoard-rescue:R_Small R65
+L Device:R_Small R65
 U 1 1 5C9F129C
 P 7750 3000
@@
 $EndComp
 $Comp
-L DFTBoard-rescue:R_Small R67
+L Device:R_Small R67
 U 1 1 5C9F48E3
 P 7750 3300
@@
 $EndComp
 $Comp
-L DFTBoard-rescue:R_Small R68
+L Device:R_Small R68
 U 1 1 5C9F4945
 P 7750 3400
@@
 DDR3_RAS#
 $Comp
-L DFTBoard-rescue:R_Small R69
+L Device:R_Small R69
 U 1 1 5C9F910F
 P 7750 3600
@@
 $EndComp
 $Comp
-L DFTBoard-rescue:R_Small R70
+L Device:R_Small R70
 U 1 1 5C9F9115
 P 7750 3700
@@
 $EndComp
 $Comp
-L DFTBoard-rescue:R_Small R71
+L Device:R_Small R71
 U 1 1 5C9F911B
 P 7750 3800
@@
 DDR3_CS#
 $Comp
-L DFTBoard-rescue:R_Small R72
+L Device:R_Small R72
 U 1 1 5CA00DBA
 P 7750 4000
@@
 $EndComp
 $Comp
-L DFTBoard-rescue:R_Small R73
+L Device:R_Small R73
 U 1 1 5CA00DC0
 P 7750 4100
@@
 Connection ~ 7850 1600
 $Comp
-L DFTBoard-rescue:R_Small R74
+L Device:R_Small R74
 U 1 1 5CA09736
 P 7900 4900
@@
 	7900 4650 7900 4800
 $Comp
-L DFTBoard-rescue:GND- #PWR0160
+L power:GND #PWR0160
 U 1 1 5CA0C7CC
 P 7900 5000
