File: LCD50.sch (KiCad schematic (older format))
At the start: 38 parts, among them Q5 IRLML2502, Q6 IRLML2502, Q7 IRLML2502, U1 xc7a50tftg256, X1 ASFLMB

Commit message: added Zynq7020 and listed all tasks outstanding
Parts:
- removed C26: .01uF, Capacitors_SMD:C_0402, symbol C_Small
- removed C27: 15pF, Capacitors_SMD:C_0402, symbol C_Small
- removed U1: xc7a50tftg256, SMD_Packages:BGA-256, symbol xc7a50tftg256
- removed X1: ASFLMB, DFTcustom:ASFLMB, symbol ASFLMB
- added U6: xc7z020clg400-, symbol DFTBoard-rescue:xc7z020clg400-
- C86: renamed from C30; symbol C_Small -> DFTBoard-rescue:C_Small-
- C87: renamed from C31; symbol C_Small -> DFTBoard-rescue:C_Small-
- C88: renamed from C34; symbol C -> DFTBoard-rescue:C-
- C89: renamed from C28; symbol C_Small -> DFTBoard-rescue:C_Small-
- C90: renamed from C29; symbol C_Small -> DFTBoard-rescue:C_Small-
- C91: renamed from C32; symbol C_Small -> DFTBoard-rescue:C_Small-
- C92: renamed from C33; symbol C_Small -> DFTBoard-rescue:C_Small-
- C93: renamed from C36; symbol C_Small -> DFTBoard-rescue:C_Small-
- C94: renamed from C37; symbol C_Small -> DFTBoard-rescue:C_Small-
- C95: renamed from C38; symbol C_Small -> DFTBoard-rescue:C_Small-
- C96: renamed from C39; symbol C_Small -> DFTBoard-rescue:C_Small-
- C97: renamed from C40; symbol C_Small -> DFTBoard-rescue:C_Small-
- C98: renamed from C41; symbol C_Small -> DFTBoard-rescue:C_Small-
- C99: renamed from C42; symbol C_Small -> DFTBoard-rescue:C_Small-
- CONN1: symbol ER-CON06HB-1 -> DFTBoard-rescue:ER-CON06HB-1-
- CONN2: symbol ER-CON50HT-1 -> DFTBoard-rescue:ER-CON50HT-1-
- D4: renamed from D2; symbol LED_RGB-RESCUE-DFTBoard -> DFTBoard-rescue:LED_RGB-RESCUE-DFTBoard-
- Q5, Q6, Q7: symbol IRLML2502 -> DFTBoard-rescue:IRLML2502-
- R28: renamed from R46; symbol R -> DFTBoard-rescue:R-
- R29: renamed from R47; symbol R -> DFTBoard-rescue:R-
- R30: renamed from R48; symbol R -> DFTBoard-rescue:R-
- R31: renamed from R43; symbol R -> DFTBoard-rescue:R-
- R32: renamed from R44; symbol R -> DFTBoard-rescue:R-
- R33: renamed from R45; symbol R -> DFTBoard-rescue:R-
- R34: renamed from R30; symbol R -> DFTBoard-rescue:R-
- R35: renamed from R31; symbol R -> DFTBoard-rescue:R-
- R36: renamed from R33; symbol R -> DFTBoard-rescue:R-
- R37: renamed from R34; symbol R -> DFTBoard-rescue:R-
- R38: renamed from R39; symbol R -> DFTBoard-rescue:R-
- R39: renamed from R40; symbol R -> DFTBoard-rescue:R-
- R40: renamed from R41; symbol R -> DFTBoard-rescue:R-
- R41: renamed from R42; symbol R -> DFTBoard-rescue:R-
Connections:
- net labels removed: CLK100MHz
- wire segments 98 -> 116
- no-connect marks 28 -> 19
Other:
- moved on the sheet: C86, C87, CONN1

Commit message: passes ERC, about to update footprints to v5 references
Parts:
- removed C88: 1uF, Capacitors_SMD:C_0603, symbol DFTBoard-rescue:C-
- removed D4: LED_RGB, DFTcustom:PLCC6-SM-RGB-LED, symbol DFTBoard-rescue:LED_RGB-RESCUE-DFTBoard-
- removed Q5, Q6, Q7: IRLML2502, TO_SOT_Packages_SMD:SOT-23, symbol DFTBoard-rescue:IRLML2502-
- removed R28, R29, R30, R31, R32: 100, Resistors_SMD:R_0402, symbol DFTBoard-rescue:R-
- removed R33: 150, Resistors_SMD:R_0402, symbol DFTBoard-rescue:R-
- added D4, D5, D6: BLUE LED, LEDs:LED_0603, symbol DFTBoard-rescue:LED-
- added Q10, Q8, Q9: IRLML2502, TO_SOT_Packages_SMD:SOT-23, symbol DFTBoard-rescue:IRLML2502-
- added R77, R79, R85: 1k, Resistors_SMD:R_0402, symbol DFTBoard-rescue:R_Small-
- added R78, R80, R86: 150, Resistors_SMD:R_0402, symbol DFTBoard-rescue:R_Small-
- U8: renamed from U6; value xc7z020clg400- -> xc7z020clg400; footprint (none) -> Package_BGA:BGA-400_21.0x21.0mm_Layout20x20_P1.0mm
- renumbered C86 to C107, C87 to C108, C89 to C109, C90 to C110, C91 to C111, C92 to C112, C93 to C113, C94 to C114, C95 to C115, C96 to C116, C97 to C117, C98 to C118, C99 to C119, R38 to R81, R39 to R82, R40 to R83, R41 to R84, R34 to R87, R35 to R88, R36 to R89, R37 to R90
Connections:
- net +5V: now also R78.2, R80.2, R86.2
- net GND: now also Q10.2 (S), Q8.2 (S), Q9.2 (S)
- net STATLED_1: now reaches U8.N17 (IO_L23P_T3_34)
- net STATLED_1: now also R79.2
- net STATLED_2: now reaches U8.P16 (IO_L24N_T3_34)
- net STATLED_2: now also R85.2
- net STATLED_0: now reaches U8.P18 (IO_L23N_T3_34)
- net STATLED_0: now also R77.2
- net I2C_SCLK renamed I2C33_SCLK
- net I2C_SDIN renamed I2C33_SDIN
- new net SLED0_D: D4.1 (K), Q8.3 (D)
- new net SLED0_G: Q8.1 (G), R77.1
- new net SLED0_R: D4.2 (A), R78.1
- new net SLED1_D: D5.1 (K), Q9.3 (D)
- new net SLED1_G: Q9.1 (G), R79.1
- new net SLED1_R: D5.2 (A), R80.1
- new net SLED2_D: D6.1 (K), Q10.3 (D)
- new net SLED2_G: Q10.1 (G), R85.1
- new net SLED2_R: D6.2 (A), R86.1
- no-connect marks 19 -> 16
Other:
- moved on the sheet: C107, C108, C109, C110, C111, C112, C113, C114, C115, C116, C117, C118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

Commit message: replacing rescue components foreal
Parts:
- U8: footprint Package_BGA:BGA-400_21.0x21.0mm_Layout20x20_P1.0mm -> DFTcustom:BGA400_0.8p_17mmx17mm
Changed lines of the file:
@@
 F 0 "U8" H 10131 -1747 60  0000 L CNN
 F 1 "xc7z020clg400" H 10131 -1853 60  0000 L CNN
-F 2 "Package_BGA:BGA-400_21.0x21.0mm_Layout20x20_P1.0mm" H 8600 700 60  0001 C CNN
+F 2 "DFTcustom:BGA400_0.8p_17mmx17mm" H 8600 700 60  0001 C CNN
 F 3 "" H 8600 700 60  0001 C CNN
 	3    8600 700

Commit message: still works, miraculously
Parts:
- C107, C108, C109, C110, C111, C112, C114, C115, C116, C117, C118, C119: footprint Capacitors_SMD:C_0603 -> Capacitor_SMD:C_0603_1608Metric; symbol DFTBoard-rescue:C_Small- -> Device:C_Small
- C113: footprint Capacitors_SMD:C_1210 -> Capacitor_SMD:C_1210_3225Metric; symbol DFTBoard-rescue:C_Small- -> Device:C_Small
- Q10, Q8, Q9: footprint TO_SOT_Packages_SMD:SOT-23 -> Package_TO_SOT_SMD:SOT-23
- R77, R78, R79, R80, R85, R86: symbol DFTBoard-rescue:R_Small- -> Device:R_Small
- R81, R82, R83, R84, R87, R88, R89, R90: symbol DFTBoard-rescue:R- -> Device:R
Connections:
- net +1.8V renamed +1V8
Changed lines of the file:
@@
 $EndDescr
 $Comp
-L DFTBoard-rescue:C_Small- C?
+L Device:C_Small C?
 U 1 1 5908520B
 P 8100 6100
@@
 F 0 "C113" H 8110 6170 50  0000 L CNN
 F 1 "47uF" H 8110 6020 50  0000 L CNN
-F 2 "Capacitors_SMD:C_1210" H 8100 6100 50  0001 C CNN
+F 2 "Capacitor_SMD:C_1210_3225Metric" H 8100 6100 50  0001 C CNN
 F 3 "" H 8100 6100 50  0001 C CNN
 F 4 "Murata Manufacturing Co Ltd" H -1000 -200 50  0001 C CNN "MFR"
@@
 $EndComp
 $Comp
-L DFTBoard-rescue:C_Small- C?
+L Device:C_Small C?
 U 1 1 59085212
 P 8350 6100
@@
 F 0 "C114" H 8360 6170 50  0000 L CNN
 F 1 "4.7uF" H 8360 6020 50  0000 L CNN
-F 2 "Capacitors_SMD:C_0603" H 8350 6100 50  0001 C CNN
+F 2 "Capacitor_SMD:C_0603_1608Metric" H 8350 6100 50  0001 C CNN
 F 3 "" H 8350 6100 50  0001 C CNN
 F 4 "Murata" H -1000 -200 50  0001 C CNN "MFR"
@@
 $EndComp
 $Comp
-L DFTBoard-rescue:C_Small- C?
+L Device:C_Small C?
 U 1 1 59085219
 P 8600 6100
@@
 F 0 "C115" H 8610 6170 50  0000 L CNN
 F 1 "4.7uF" H 8610 6020 50  0000 L CNN
-F 2 "Capacitors_SMD:C_0603" H 8600 6100 50  0001 C CNN
+F 2 "Capacitor_SMD:C_0603_1608Metric" H 8600 6100 50  0001 C CNN
 F 3 "" H 8600 6100 50  0001 C CNN
 F 4 "Murata" H -1000 -200 50  0001 C CNN "MFR"
@@
 $EndComp
 $Comp
-L DFTBoard-rescue:C_Small- C?
+L Device:C_Small C?
 U 1 1 59085220
 P 8850 6100
@@
 F 0 "C116" H 8860 6170 50  0000 L CNN
 F 1 ".47uF" H 8860 6020 50  0000 L CNN
-F 2 "Capacitors_SMD:C_0603" H 8850 6100 50  0001 C CNN
+F 2 "Capacitor_SMD:C_0603_1608Metric" H 8850 6100 50  0001 C CNN
 F 3 "" H 8850 6100 50  0001 C CNN
 F 4 "Murata" H -1000 -200 50  0001 C CNN "MFR"
@@
 $EndComp
 $Comp
-L DFTBoard-rescue:C_Small- C?
+L Device:C_Small C?
 U 1 1 59085227
 P 9100 6100
@@
 F 0 "C117" H 9110 6170 50  0000 L CNN
 F 1 ".47uF" H 9110 6020 50  0000 L CNN
-F 2 "Capacitors_SMD:C_0603" H 9100 6100 50  0001 C CNN
+F 2 "Capacitor_SMD:C_0603_1608Metric" H 9100 6100 50  0001 C CNN
 F 3 "" H 9100 6100 50  0001 C CNN
 F 4 "Murata" H -1000 -200 50  0001 C CNN "MFR"
@@
 $EndComp
 $Comp
-L DFTBoard-rescue:C_Small- C?
+L Device:C_Small C?
 U 1 1 5908522E
 P 9350 6100
@@
 F 0 "C118" H 9360 6170 50  0000 L CNN
 F 1 ".47uF" H 9360 6020 50  0000 L CNN
-F 2 "Capacitors_SMD:C_0603" H 9350 6100 50  0001 C CNN
+F 2 "Capacitor_SMD:C_0603_1608Metric" H 9350 6100 50  0001 C CNN
 F 3 "" H 9350 6100 50  0001 C CNN
 F 4 "Murata" H -1000 -200 50  0001 C CNN "MFR"
@@
 $EndComp
 $Comp
-L DFTBoard-rescue:C_Small- C?
+L Device:C_Small C?
 U 1 1 59085235
 P 9600 6100
@@
 F 0 "C119" H 9610 6170 50  0000 L CNN
 F 1 ".47uF" H 9610 6020 50  0000 L CNN
-F 2 "Capacitors_SMD:C_0603" H 9600 6100 50  0001 C CNN
+F 2 "Capacitor_SMD:C_0603_1608Metric" H 9600 6100 50  0001 C CNN
 F 3 "" H 9600 6100 50  0001 C CNN
 F 4 "Murata" H -1000 -200 50  0001 C CNN "MFR"
@@
 $EndComp
 $Comp
-L DFTBoard-rescue:GND- #PWR?
+L power:GND #PWR?
 U 1 1 5908523C
 P 8850 6400
@@
 $EndComp
 $Comp
-L DFTBoard-rescue:GND- #PWR?
+L power:GND #PWR?
 U 1 1 598A88E7
 P 6600 1100
@@
 $EndComp
 $Comp
-L DFTBoard-rescue:GND- #PWR?
+L power:GND #PWR?
 U 1 1 598ADA0E
 P 6600 1700
@@
 $EndComp
 $Comp
-L DFTBoard-rescue:GND- #PWR?
+L power:GND #PWR?
 U 1 1 598B6836
 P 6500 5900
@@
 $EndComp
 $Comp
-L DFTBoard-rescue:+1.8V- #PWR?
+L power:+1V8 #PWR?
 U 1 1 598B6CF5
 P 8600 5900
@@
 $EndComp
 $Comp
-L DFTBoard-rescue:+3.3V- #PWR?
+L power:+3V3 #PWR?
 U 1 1 598B98DD
 P 7400 1400
@@
 $EndComp
 $Comp
-L DFTBoard-rescue:+1.8V- #PWR?
+L power:+1V8 #PWR?
 U 1 1 598BA87D
 P 7500 2000
@@
 $EndComp
 $Comp
-L DFTBoard-rescue:C_Small- C?
+L Device:C_Small C?
 U 1 1 598BDB12
 P 7200 1550
@@
 F 0 "C110" H 7210 1620 50  0000 L CNN
 F 1 "4.7uF" H 7210 1470 50  0000 L CNN
-F 2 "Capacitors_SMD:C_0603" H 7200 1550 50  0001 C CNN
+F 2 "Capacitor_SMD:C_0603_1608Metric" H 7200 1550 50  0001 C CNN
 F 3 "" H 7200 1550 50  0001 C CNN
 F 4 "Murata" H -1000 -200 50  0001 C CNN "MFR"
@@
 $EndComp
 $Comp
-L DFTBoard-rescue:C_Small- C?
+L Device:C_Small C?
 U 1 1 598BDB19
 P 7000 1550
@@
 F 0 "C109" H 7010 1620 50  0000 L CNN
 F 1 ".1uF" H 7010 1470 50  0000 L CNN
-F 2 "Capacitors_SMD:C_0603" H 7000 1550 50  0001 C CNN
+F 2 "Capacitor_SMD:C_0603_1608Metric" H 7000 1550 50  0001 C CNN
 F 3 "" H 7000 1550 50  0001 C CNN
 F 4 "Murata" H -1000 -200 50  0001 C CNN "MFR"
@@
 $EndComp
 $Comp
-L DFTBoard-rescue:C_Small- C?
+L Device:C_Small C?
 U 1 1 598BE44E
 P 7400 2150
@@
 F 0 "C112" H 7410 2220 50  0000 L CNN
 F 1 "4.7uF" H 7410 2070 50  0000 L CNN
-F 2 "Capacitors_SMD:C_0603" H 7400 2150 50  0001 C CNN
+F 2 "Capacitor_SMD:C_0603_1608Metric" H 7400 2150 50  0001 C CNN
 F 3 "" H 7400 2150 50  0001 C CNN
 F 4 "Murata" H -1000 -200 50  0001 C CNN "MFR"
@@
 $EndComp
 $Comp
-L DFTBoard-rescue:C_Small- C?
+L Device:C_Small C?
 U 1 1 598BE454
 P 7200 2150
@@
 F 0 "C111" H 7210 2220 50  0000 L CNN
 F 1 ".1uF" H 7210 2070 50  0000 L CNN
-F 2 "Capacitors_SMD:C_0603" H 7200 2150 50  0001 C CNN
+F 2 "Capacitor_SMD:C_0603_1608Metric" H 7200 2150 50  0001 C CNN
 F 3 "" H 7200 2150 50  0001 C CNN
 F 4 "Murata" H -1000 -200 50  0001 C CNN "MFR"
@@
 $EndComp
 $Comp
-L DFTBoard-rescue:GND- #PWR?
+L power:GND #PWR?
 U 1 1 598BEE0D
 P 7100 1750
@@
 $EndComp
 $Comp
-L DFTBoard-rescue:GND- #PWR?
+L power:GND #PWR?
 U 1 1 598BEE7B
 P 7300 2350
@@
 $EndComp
 $Comp
-L DFTBoard-rescue:R- R?
+L Device:R R?
 U 1 1 598CC6B6
 P 6500 5500
@@
 $EndComp
 $Comp
-L DFTBoard-rescue:R- R?
+L Device:R R?
 U 1 1 598CC81A
 P 6500 5600
@@
 $EndComp
 $Comp
-L DFTBoard-rescue:R- R?
+L Device:R R?
 U 1 1 598CCA98
 P 6500 5700
@@
 $EndComp
 $Comp
-L DFTBoard-rescue:R- R?
+L Device:R R?
 U 1 1 598CCAAA
 P 6500 5800
@@
 $EndComp
 $Comp
-L DFTBoard-rescue:+3.3V- #PWR?
+L power:+3V3 #PWR?
 U 1 1 598CDBCB
 P 6900 5650
@@
 $EndComp
 $Comp
-L DFTBoard-rescue:GND- #PWR?
+L power:GND #PWR?
 U 1 1 598F040F
 P 4550 1100
@@
 $EndComp
 $Comp
-L DFTBoard-rescue:+3.3V- #PWR?
+L power:+3V3 #PWR?
 U 1 1 598F1F44
 P 4100 1600
@@
 $EndComp
 $Comp
-L DFTBoard-rescue:C_Small- C?
+L Device:C_Small C?
 U 1 1 598FD60E
 P 4400 1800
@@
 F 0 "C108" H 4410 1870 50  0000 L CNN
 F 1 "4.7uF" H 4410 1720 50  0000 L CNN
-F 2 "Capacitors_SMD:C_0603" H 4400 1800 50  0001 C CNN
+F 2 "Capacitor_SMD:C_0603_1608Metric" H 4400 1800 50  0001 C CNN
 F 3 "" H 4400 1800 50  0001 C CNN
 F 4 "Murata" H -200 -500 50  0001 C CNN "MFR"
@@
 $EndComp
 $Comp
-L DFTBoard-rescue:C_Small- C?
+L Device:C_Small C?
 U 1 1 598FD614
 P 4200 1800
@@
 F 0 "C107" H 4210 1870 50  0000 L CNN
 F 1 ".1uF" H 4210 1720 50  0000 L CNN
-F 2 "Capacitors_SMD:C_0603" H 4200 1800 50  0001 C CNN
+F 2 "Capacitor_SMD:C_0603_1608Metric" H 4200 1800 50  0001 C CNN
 F 3 "" H 4200 1800 50  0001 C CNN
 F 4 "Murata" H -200 -500 50  0001 C CNN "MFR"
@@
 $EndComp
 $Comp
-L DFTBoard-rescue:GND- #PWR?
+L power:GND #PWR?
 U 1 1 598FDD2A
 P 4300 2100
@@
 $EndComp
 $Comp
-L DFTBoard-rescue:+1.8V- #PWR?
+L power:+1V8 #PWR?
 U 1 1 598CFD34
 P 4400 3600
@@
 $EndComp
 $Comp
-L DFTBoard-rescue:GND- #PWR?
+L power:GND #PWR?
 U 1 1 598D049B
 P 4150 3600
@@
 $EndComp
 $Comp
-L DFTBoard-rescue:R- R?
+L Device:R R?
 U 1 1 598E0C58
 P 4100 3300
@@
 $EndComp
 $Comp
-L DFTBoard-rescue:R- R?
+L Device:R R?
 U 1 1 598E0CC1
 P 4200 3300
@@
 $EndComp
 $Comp
-L DFTBoard-rescue:R- R?
+L Device:R R?
 U 1 1 598E0E36
 P 4350 3300
@@
 $EndComp
 $Comp
-L DFTBoard-rescue:R- R?
+L Device:R R?
 U 1 1 598E0EDE
 P 4450 3300
@@
 F 0 "Q9" H 3400 5651 40  0000 R CNN
 F 1 "IRLML2502" H 3400 5950 40  0000 R CNN
-F 2 "TO_SOT_Packages_SMD:SOT-23" H 3270 5902 29  0001 C CNN
+F 2 "Package_TO_SOT_SMD:SOT-23" H 3270 5902 29  0001 C CNN
 F 3 "" H 3400 5800 60  0001 C CNN
 F 4 "Infineon Technologies AG" H 1450 -1250 50  0001 C CNN "MFR"
@@
 F 0 "Q8" H 1750 5651 40  0000 R CNN
 F 1 "IRLML2502" H 1750 5950 40  0000 R CNN
-F 2 "TO_SOT_Packages_SMD:SOT-23" H 1620 5902 29  0001 C CNN
+F 2 "Package_TO_SOT_SMD:SOT-23" H 1620 5902 29  0001 C CNN
 F 3 "" H 1750 5800 60  0001 C CNN
 F 4 "Infineon Technologies AG" H -200 550 50  0001 C CNN "MFR"
@@
 $EndComp
 $Comp
-L DFTBoard-rescue:GND- #PWR?
+L power:GND #PWR?
 U 1 1 5CA0A768
 P 3500 6050
@@
 $EndComp
 $Comp
-L DFTBoard-rescue:GND- #PWR?
+L power:GND #PWR?
 U 1 1 5CA0A76E
 P 1850 6050
@@
 $EndComp
 $Comp
-L DFTBoard-rescue:R_Small- R?
+L Device:R_Small R?
 U 1 1 5CA0A779
 P 3050 5850
@@
 $EndComp
 $Comp
-L DFTBoard-rescue:R_Small- R?
+L Device:R_Small R?
 U 1 1 5CA0A785
 P 1400 5850
@@
 $EndComp
 $Comp
-L DFTBoard-rescue:R_Small- R?
+L Device:R_Small R?
 U 1 1 5CA0A7A9
 P 3500 4900
@@
 $EndComp
 $Comp
-L DFTBoard-rescue:R_Small- R?
+L Device:R_Small R?
 U 1 1 5CA0A7B5
 P 1850 4900
@@
 $EndComp
 $Comp
-L DFTBoard-rescue:+5V- #PWR?
+L power:+5V #PWR?
 U 1 1 5CA0A7BC
 P 3500 4700
@@
 $EndComp
 $Comp
-L DFTBoard-rescue:+5V- #PWR?
+L power:+5V #PWR?
 U 1 1 5CA0A7C2
 P 1850 4750
@@
 F 0 "Q10" H 4900 5651 40  0000 R CNN
 F 1 "IRLML2502" H 4900 5950 40  0000 R CNN
-F 2 "TO_SOT_Packages_SMD:SOT-23" H 4770 5902 29  0001 C CNN
+F 2 "Package_TO_SOT_SMD:SOT-23" H 4770 5902 29  0001 C CNN
 F 3 "" H 4900 5800 60  0001 C CNN
 F 4 "Infineon Technologies AG" H 2950 550 50  0001 C CNN "MFR"
@@
 $EndComp
 $Comp
-L DFTBoard-rescue:GND- #PWR?
+L power:GND #PWR?
 U 1 1 5CA0A7E3
 P 5000 6050
@@
 $EndComp
 $Comp
-L DFTBoard-rescue:R_Small- R?
+L Device:R_Small R?
 U 1 1 5CA0A7EE
 P 4550 5850
@@
 $EndComp
 $Comp
-L DFTBoard-rescue:R_Small- R?
+L Device:R_Small R?
 U 1 1 5CA0A806
 P 5000 4900
@@
 $EndComp
 $Comp
-L DFTBoard-rescue:+5V- #PWR?
+L power:+5V #PWR?
 U 1 1 5CA0A80D
 P 5000 4750

Commit message: random updates
Parts:
- removed U8: xc7z020clg400, DFTcustom:BGA400_0.8p_17mmx17mm, symbol DFTBoard-rescue:xc7z020clg400-
- added U20: xc7z020clg484, DFTcustom:BGA-484_19.0x19.0mm_Layout22x22_P0.80mm_dia0.40mm, symbol xilinx7:xc7z020clg484
- C107, C108, C109, C110, C111, C112, C114, C115, C116, C117, C118, C119: footprint Capacitor_SMD:C_0603_1608Metric -> Capacitor_SMD:C_0402_1005Metric
- D4, D5, D6: footprint LEDs:LED_0603 -> Capacitor_SMD:C_0603_1608Metric
- R77, R78, R79, R80, R81, R82, R83, R84, R85, R86, R87, R88, R89, R90: footprint Resistors_SMD:R_0402 -> Resistor_SMD:R_0402_1005Metric
Connections:
- net +1V8: now also U20.AA10 (VCCO_13[7]), U20.AB3 (VCCO_13[7]), U20.T5 (VCCO_13[7]), U20.U8 (VCCO_13[7]), U20.V11 (VCCO_13[7]), U20.W4 (VCCO_13[7]), U20.Y7 (VCCO_13[7])
- net LCD_CS: now also U20.W6 (IO_L24P_T3_13)
- net LCD_D0: now also U20.U4 (IO_L20N_T3_13)
- net LCD_D1: now also U20.AB7 (IO_L17P_T2_13)
- net LCD_D10: now also U20.AB10 (IO_L9P_T1_DQS_13)
- net LCD_D11: now also U20.Y11 (IO_L10P_T1_13)
- net LCD_D12: now also U20.Y8 (IO_L12N_T1_MRCC_13)
- net LCD_D13: now also U20.U9 (IO_L6N_T0_VREF_13)
- net LCD_D14: now also U20.AA9 (IO_L11P_T1_SRCC_13)
- net LCD_D15: now also U20.U10 (IO_L6P_T0_13)
- net LCD_D16: now also U20.AB9 (IO_L9N_T1_DQS_13)
- net LCD_D17: now also U20.AB12 (IO_L7N_T1_13)
- net LCD_D2: now also U20.AB6 (IO_L17N_T2_13)
- net LCD_D3: now also U20.AB4 (IO_L16N_T2_13)
- net LCD_D4: now also U20.AA6 (IO_L14N_T2_SRCC_13)
- net LCD_D5: now also U20.AB2 (IO_L15P_T2_DQS_13)
- net LCD_D6: now also U20.AA7 (IO_L14P_T2_SRCC_13)
- net LCD_D7: now also U20.Y10 (IO_L10N_T1_13)
- net LCD_D8: now also U20.AB1 (IO_L15N_T2_DQS_13)
- net LCD_D9: now also U20.AA8 (IO_L11N_T1_SRCC_13)
- net LCD_DorI: now also U20.V5 (IO_L21P_T3_DQS_13)
- net LCD_IM0: now also U20.V8 (IO_L2P_T0_13)
- net LCD_IM1: now also U20.U11 (IO_L5N_T0_13)
- net LCD_IM2: now also U20.W11 (IO_L3P_T0_DQS_13)
- net LCD_IM3: now also U20.W10 (IO_L3N_T0_DQS_13)
- net LCD_READ: now also U20.T6 (IO_L19N_T3_VREF_13)
- net LCD_RST: now also U20.V12 (IO_L4P_T0_13)
- net LCD_SDI: now also U20.T4 (IO_L20P_T3_13)
- net LCD_SDO: now also U20.V4 (IO_L21N_T3_DQS_13)
- net LCD_TE: now also U20.U6 (IO_L22P_T3_13)
- net LCD_WRITE: now also U20.U5 (IO_L22N_T3_13)
- net RGB_DE: now also U20.AA11 (IO_L8P_T1_13)
- net RGB_DOTCLK: now also U20.AB11 (IO_L8N_T1_13)
- net RGB_HSYNC: now also U20.AA12 (IO_L7P_T1_13)
- net RGB_VSYNC: now also U20.W12 (IO_L4N_T0_13)
- net STATLED_0: now also U20.W7 (IO_L23N_T3_13)
- net STATLED_1: now also U20.V7 (IO_L23P_T3_13)
- net STATLED_2: now also U20.W5 (IO_L24N_T3_13)
- net TEMPO_LED: now also U20.V9 (IO_L1N_T0_13)
- net I2C33_SDIN renamed I2C33_SDA
Other:
- moved on the sheet: C107, C108, C109, C110, C111, C112, C113, C114, C115, C116, C117, C118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
